File: engine-control-unit_prototype/ECU_COM.kicad_sch (KiCad schematic)
At the start: 4 parts, among them J2 DE9_Pins_MountingHoles, U3 TCAN337G

Commit message: Added power circuitry without components values
Parts:
- renumbered C44 to C46, J2 to J8, R2 to R13, U3 to U5
Changed lines of the file:
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@@
 		(on_board yes)
 		(dnp no)
-		(property "Reference" "#PWR059"
+		(property "Reference" "#PWR074"
 			(at 69.85 41.91 0)
 			(effects
@@
 			(project "engine-control-unit_prototype"
 				(path "/4da294f1-7505-49eb-91fe-5b5cfad6e8fb/2469e973-1fee-44cf-8019-cdd458641741"
-					(reference "#PWR059")
+					(reference "#PWR074")
 					(unit 1)
 				)
@@
 		(on_board yes)
 		(dnp no)
-		(property "Reference" "R2"
+		(property "Reference" "R13"
 			(at 46.99 62.23 90)
 			(effects
@@
 			(project "engine-control-unit_prototype"
 				(path "/4da294f1-7505-49eb-91fe-5b5cfad6e8fb/2469e973-1fee-44cf-8019-cdd458641741"
-					(reference "R2")
+					(reference "R13")
 					(unit 1)
 				)
@@
 		(dnp no)
 		(fields_autoplaced yes)
-		(property "Reference" "U3"
+		(property "Reference" "U5"
 			(at 71.9933 40.64 0)
 			(effects
@@
 			(project "engine-control-unit_prototype"
 				(path "/4da294f1-7505-49eb-91fe-5b5cfad6e8fb/2469e973-1fee-44cf-8019-cdd458641741"
-					(reference "U3")
+					(reference "U5")
 					(unit 1)
 				)
@@
 		(dnp no)
 		(fields_autoplaced yes)
-		(property "Reference" "J2"
+		(property "Reference" "J8"
 			(at 161.29 66.0399 0)
 			(effects
@@
 			(project "engine-control-unit_prototype"
 				(path "/4da294f1-7505-49eb-91fe-5b5cfad6e8fb/2469e973-1fee-44cf-8019-cdd458641741"
-					(reference "J2")
+					(reference "J8")
 					(unit 1)
 				)
@@
 		(on_board yes)
 		(dnp no)
-		(property "Reference" "#PWR058"
+		(property "Reference" "#PWR075"
 			(at 86.36 52.07 0)
 			(effects
@@
 			(project "engine-control-unit_prototype"
 				(path "/4da294f1-7505-49eb-91fe-5b5cfad6e8fb/2469e973-1fee-44cf-8019-cdd458641741"
-					(reference "#PWR058")
+					(reference "#PWR075")
 					(unit 1)
 				)
@@
 		(dnp no)
 		(fields_autoplaced yes)
-		(property "Reference" "C44"
+		(property "Reference" "C46"
 			(at 90.17 40.6399 0)
 			(effects
@@
 			(project "engine-control-unit_prototype"
 				(path "/4da294f1-7505-49eb-91fe-5b5cfad6e8fb/2469e973-1fee-44cf-8019-cdd458641741"
-					(reference "C44")
+					(reference "C46")
 					(unit 1)
 				)
@@
 		(on_board yes)
 		(dnp no)
-		(property "Reference" "#PWR057"
+		(property "Reference" "#PWR078"
 			(at 148.59 95.25 0)
 			(effects
@@
 			(project "engine-control-unit_prototype"
 				(path "/4da294f1-7505-49eb-91fe-5b5cfad6e8fb/2469e973-1fee-44cf-8019-cdd458641741"
-					(reference "#PWR057")
+					(reference "#PWR078")
 					(unit 1)
 				)
@@
 		(on_board yes)
 		(dnp no)
-		(property "Reference" "#PWR054"
+		(property "Reference" "#PWR076"
 			(at 69.85 69.85 0)
 			(effects
@@
 			(project "engine-control-unit_prototype"
 				(path "/4da294f1-7505-49eb-91fe-5b5cfad6e8fb/2469e973-1fee-44cf-8019-cdd458641741"
-					(reference "#PWR054")
+					(reference "#PWR076")
 					(unit 1)
 				)
@@
 		(on_board yes)
 		(dnp no)
-		(property "Reference" "#PWR060"
+		(property "Reference" "#PWR077"
 			(at 49.53 72.39 0)
 			(effects
@@
 			(project "engine-control-unit_prototype"
 				(path "/4da294f1-7505-49eb-91fe-5b5cfad6e8fb/2469e973-1fee-44cf-8019-cdd458641741"
-					(reference "#PWR060")
-					(unit 1)
-				)
+					(reference "#PWR077")
+					(unit 1)
+				)
