File: engine-control-unit_prototype/ECU_SMPS.kicad_sch (KiCad schematic)
At the start: 18 parts

Commit message: Added power circuitry without components values
Parts:
- renumbered C21 to C67, C33 to C68, C40 to C69, C41 to C70, C42 to C71, C19 to C72, C20 to C73, C22 to C74, JP9 to JP10, JP10 to JP11, JP11 to JP12, JP7 to JP5, JP5 to JP6, JP8 to JP7, JP4 to JP8, JP6 to JP9, L2 to L3, L1 to L4

Commit message: Removed bloat libraries Changed symbols for Sirius custom library Changed layout for one page
Parts:
- removed C67: 4.7u ESR < 100m, symbol Device:C
- removed C68, C69: 2.2u ESR < 100m, symbol Device:C
- removed C70, C71: 4.7u, symbol Device:C
- removed C72: 220p, symbol Device:C
- removed C73, C74: 10u ESR < 20m, symbol Device:C
- removed JP10, JP11, JP12, JP6, JP7: SMPS, symbol Jumper:SolderJumper_2_Open
- removed JP5, JP8, JP9: LDO, symbol Jumper:SolderJumper_2_Open
- removed L3: FBMJ1608HM180NTR, symbol Device:L_Ferrite
- removed L4: 2.2u, symbol Device:L
Other:
- note removed: "(1)"
- note removed: "(1) Jumpers pour choix entre SMPS direct ou SMPS externe avec LDO par SMPS"
- note removed: "(2)"
- note removed: "(2) Bead utilisé dans eval board"
- note removed: "(3)"
- note removed: "(3) Choix des condensateurs pour SMPS [p.103, p.110 | stm32h757ai.pdf]"
- note removed: "(4)"
- note removed: "(4) Datasheet dit 4.7uF, mais eval board met 10uF"
- note removed: "Datasheet STM32H747"
- note removed: "Placer proche L1"
- note removed: "Schematic Eval board STM32H7X7"
