File: engine-control-unit_prototype/engine-control-unit_prototype.kicad_pcb (KiCad board)
At the start: 2 copper layers, 324 parts, among them J1 JTAG, J2 USB_C_Receptacle_USB2.0_man, J3 Micro_SD_Card_Det1, U1 USBLC6-2SC6, U11 LT3042xMSE, U12 ADS131M04xPW, U13 INA219AxD, U14 LT3042xMSE, U3 INA826, U6 INA219AxD, U7 STM32H747II, U8 INA219AxD

Commit message: Started layout Added some footprints
Parts:
- removed C32, C65: C, Capacitor_SMD:C_0603_1608Metric
- removed C33: 10nF, Capacitor_SMD:C_0402_1005Metric
- removed C34: 10u, Capacitor_SMD:C_0603_1608Metric
- removed F1: Polyfuse, Fuse:Fuse_0603_1608Metric_Pad1.05x0.95mm_HandSolder
- removed the R10 at (106.1, 98.2)
- removed the R100 at (52.8, 147.0)
- removed the R101 at (52.8, 148.8)
- removed the R102 at (52.8, 150.5)
- removed the R11 at (110.1, 85.7)
- removed the R12 at (110.1, 88.2)
- removed the R16 at (174.8, 84.5)
- removed the R17 at (174.8, 86.5)
- removed the R18 at (174.8, 88.5)
- removed the R19 at (174.8, 90.5)
- removed the R2 at (47.8, 55.8)
- removed the R20 at (174.8, 92.4)
- removed the R21 at (177.7, 80.5)
- removed the R22 at (67.6, 83.2)
- removed R228, R229: 1k, Resistor_SMD:R_0402_1005Metric
- removed the R23 at (67.6, 85.8)
- removed the R24 at (177.7, 82.5)
- removed the R25 at (67.6, 88.3)
- removed the R26 at (67.6, 90.8)
- removed the R27 at (67.6, 93.3)
- removed the R28 at (67.6, 95.8)
- removed the R3 at (102.1, 76.4)
- removed the R30 at (67.6, 98.3)
- removed the R31 at (67.6, 100.8)
- removed the R32 at (177.7, 84.5)
- removed the R33 at (177.7, 86.5)
- removed the R34 at (43.0, 59.0)
- removed the R35 at (43.0, 60.0)
- removed the R36 at (39.7, 56.0)
- removed the R37 at (71.6, 80.7)
- removed the R38 at (42.5, 58.0)
- removed the R39 at (39.7, 59.5)
- removed the R40 at (71.6, 83.2)
- removed the R42 at (47.8, 56.8)
- removed the R43 at (38.5, 74.8)
- removed the R44 at (38.5, 76.5)
- removed the R45 at (38.5, 78.2)
- removed the R46 at (38.5, 80.0)
- removed the R47 at (38.5, 81.8)
- removed the R48 at (38.5, 83.5)
- removed the R49 at (138.5, 49.2)
- removed the R5 at (113.4, 99.7)
- removed the R51 at (141.0, 49.2)
- removed the R52 at (143.2, 49.2)
- removed the R53 at (145.0, 49.2)
- removed the R54 at (146.2, 49.2)
- removed the R55 at (71.6, 85.8)
- removed the R56 at (71.6, 88.3)
- removed the R57 at (71.6, 90.8)
- removed the R58 at (71.6, 93.3)
- removed the R59 at (71.6, 95.8)
- removed the R61 at (71.6, 98.3)
- removed the R62 at (147.5, 49.2)
- removed the R63 at (71.6, 100.8)
- removed the R64 at (73.2, 76.5)
- removed the R65 at (98.6, 19.0)
- removed the R66 at (98.6, 21.5)
- removed the R68 at (110.1, 90.7)
- removed the R69 at (110.1, 93.2)
- removed the R70 at (106.1, 68.9)
- removed the R71 at (88.5, 140.6)
- removed the R72 at (88.5, 143.1)
- removed the R73 at (88.5, 145.6)
- removed the R74 at (92.5, 125.5)
- removed the R75 at (92.5, 128.0)
- removed the R76 at (92.5, 130.5)
- removed the R77 at (106.5, 78.5)
- removed the R78 at (106.5, 80.3)
- removed the R8 at (113.4, 103.2)
- removed the R81 at (106.1, 71.4)
- removed the R82 at (106.1, 73.9)
- removed the R83 at (121.3, 63.6)
- removed the R84 at (121.3, 65.6)
- removed the R85 at (121.3, 67.6)
- removed the R86 at (121.3, 69.6)
- removed the R87 at (121.3, 71.6)
- removed the R88 at (124.2, 63.6)
- removed the R89 at (75.6, 83.2)
- removed the R9 at (106.1, 95.7)
- removed the R90 at (75.6, 85.8)
- removed the R91 at (75.6, 88.3)
- removed the R92 at (75.6, 90.8)
- removed the R93 at (124.2, 65.6)
- removed the R94 at (124.2, 67.6)
- removed the R97 at (52.8, 141.8)
- removed the R98 at (52.8, 143.5)
- removed the R99 at (52.8, 145.2)
- removed the U1 at (135.8, 91.2)
- removed U13: INA219AxD, Package_SO:SOIC-8_3.9x4.9mm_P1.27mm
- removed U14: LT3042xMSE, Package_SO:MSOP-10-1EP_3x3mm_P0.5mm_EP1.68x1.88mm
- added C100: C, Capacitor_SMD:C_0402_1005Metric, F.Cu at (123.0, 155.5)
- added C101: C, Capacitor_SMD:C_1206_3216Metric, F.Cu at (90.0, 164.5)
- added C102: C, Capacitor_SMD:C_0402_1005Metric, F.Cu at (127.0, 155.5)
- added C103: 100p, Capacitor_SMD:C_0402_1005Metric, F.Cu at (131.0, 160.5)
- added C104: ?, Capacitor_SMD:C_0402_1005Metric, F.Cu at (131.0, 159.5)
- added C105: C, Capacitor_SMD:C_0603_1608Metric, F.Cu at (127.0, 162.2)
- added C106: C, Capacitor_SMD:C_1206_3216Metric, F.Cu at (127.5, 164.5)
- added C27: 2.2u ESR < 600m, Capacitor_SMD:C_0603_1608Metric, F.Cu at (261.3, 20.3)
- added C31: 10u, Capacitor_SMD:C_0603_1608Metric, F.Cu at (157.8, 158.0)
- added C45: C, Capacitor_SMD:C_1206_3216Metric, F.Cu at (128.8, 184.5)
- added C58: 100n, Capacitor_SMD:C_0402_1005Metric, F.Cu at (170.3, 52.6)
- added C59: ?, Capacitor_SMD:C_0402_1005Metric, F.Cu at (280.5, 13.1)
- added C90: 0u1, Capacitor_SMD:C_0402_1005Metric, F.Cu at (276.5, 66.2)
- added C91: 0u1, Capacitor_SMD:C_0402_1005Metric, F.Cu at (276.5, 68.2)
- added C95: ?, Capacitor_SMD:C_0402_1005Metric, F.Cu at (93.5, 159.5)
- added C96: C, Capacitor_SMD:C_0603_1608Metric, F.Cu at (89.5, 162.2)
- added C97: 4u7, Capacitor_SMD:C_0603_1608Metric, F.Cu at (261.3, 27.8)
- added C98: C, Capacitor_SMD:C_0603_1608Metric, F.Cu at (85.5, 162.2)
- added C99: C, Capacitor_SMD:C_0402_1005Metric, F.Cu at (83.5, 160.0)
- added D10: BAV99, Package_TO_SOT_SMD:SOT-23, F.Cu at (291.8, 50.1)
- added D11: BAV99, Package_TO_SOT_SMD:SOT-23, F.Cu at (291.8, 54.6)
- added D3: VDD_10V, LED_SMD:LED_0603_1608Metric, F.Cu at (129.8, 32.0)
- added D7: DNF, Package_TO_SOT_SMD:SOT-23-3, F.Cu at (193.7, 49.6)
- added D9: 6.4V, Diode_SMD:D_0603_1608Metric_Pad1.05x0.95mm_HandSolder, F.Cu at (162.4, 42.4)
- added F2: Polyfuse, Fuse:Fuse_0603_1608Metric_Pad1.05x0.95mm_HandSolder, F.Cu at (162.4, 45.0)
- added IC1: TPS259573DSGR, Package_SON:WSON-8-1EP_2x2mm_P0.5mm_EP0.9x1.6mm, F.Cu at (28.9, 88.5)
- added J10: I2C, Connector_PinSocket_2.54mm:PinSocket_1x04_P2.54mm_Vertical, F.Cu at (171.2, 39.8)
- added J11: CANFD, Connector_Dsub:DSUB-9_Pins_Horizontal_P2.77x2.84mm_EdgePinOffset7.70mm_Housed_MountingHolesOffset9.12mm, F.Cu at (175.7, 19.5)
- added J12: ADXL345, Connector_PinSocket_2.54mm:PinSocket_1x09_P2.54mm_Vertical, F.Cu at (162.5, 18.5)
- added J13: MAG_CONN_1, Connector_PinSocket_2.54mm:PinSocket_1x04_P2.54mm_Vertical, F.Cu at (175.8, 39.8)
- added J14: MAG_CONN_2, Connector_PinSocket_2.54mm:PinSocket_1x04_P2.54mm_Vertical, F.Cu at (180.4, 39.8)
- added J16: USB_C_Receptacle_USB2.0_man, Connector_USB:USB_C_Receptacle_GCT_USB4105-xx-A_16P_TopMnt_Horizontal, F.Cu at (188.5, 42.7)
- added J18: VREF, Connector_PinHeader_2.54mm:PinHeader_1x01_P2.54mm_Vertical, F.Cu at (257.9, 136.4)
- added J19: PT1, Connector_PinSocket_2.54mm:PinSocket_1x04_P2.54mm_Vertical, F.Cu at (268.2, 21.4)
- added J20: PT2, Connector_PinSocket_2.54mm:PinSocket_1x04_P2.54mm_Vertical, F.Cu at (272.8, 21.4)
- added J21: PT3, Connector_PinSocket_2.54mm:PinSocket_1x04_P2.54mm_Vertical, F.Cu at (277.4, 21.4)
- added J22: PT4, Connector_PinSocket_2.54mm:PinSocket_1x04_P2.54mm_Vertical, F.Cu at (282.0, 21.4)
- added J23: PT5, Connector_PinSocket_2.54mm:PinSocket_1x04_P2.54mm_Vertical, F.Cu at (286.6, 21.4)
- added J24: HEATER_IPA, Connector_PinSocket_2.54mm:PinSocket_1x02_P2.54mm_Vertical, F.Cu at (268.2, 67.5)
- added J25: HEATER_NOS, Connector_PinSocket_2.54mm:PinSocket_1x02_P2.54mm_Vertical, F.Cu at (272.8, 67.5)
- added J26: VALVE_IPA, Connector_PinSocket_2.54mm:PinSocket_1x03_P2.54mm_Vertical, F.Cu at (286.0, 65.6)
- added J27: VALVE_NOS, Connector_PinSocket_2.54mm:PinSocket_1x03_P2.54mm_Vertical, F.Cu at (290.6, 65.6)
- added J28: NOS ENCODER, Connector_PinSocket_2.54mm:PinSocket_1x06_P2.54mm_Vertical, F.Cu at (268.2, 50.2)
- added J30: IPA ENCODER, Connector_PinSocket_2.54mm:PinSocket_1x06_P2.54mm_Vertical, F.Cu at (272.8, 50.2)
- added J31: VCTR_CONN, Connector_PinSocket_2.54mm:PinSocket_1x06_P2.54mm_Vertical, F.Cu at (277.4, 50.2)
- added J4: PORT_A, Connector_PinSocket_2.54mm:PinSocket_1x16_P2.54mm_Vertical, F.Cu at (243.2, 21.4)
- added J5: PORT_B, Connector_PinSocket_2.54mm:PinSocket_1x16_P2.54mm_Vertical, F.Cu at (247.8, 21.4)
- added J6: PORT_D, Connector_PinSocket_2.54mm:PinSocket_1x16_P2.54mm_Vertical, F.Cu at (252.4, 21.4)
- added J7: PORT_C, Connector_PinSocket_2.54mm:PinSocket_1x16_P2.54mm_Vertical, F.Cu at (257.0, 21.4)
- added J8: 2S_18650, Connector_PinSocket_2.54mm:PinSocket_1x02_P2.54mm_Vertical, F.Cu at (154.2, 18.5)
- added J9: EXT_BATT, Connector_PinSocket_2.54mm:PinSocket_1x01_P2.54mm_Vertical, F.Cu at (29.5, 163.3)
- added JP1: BATT, Connector_PinSocket_2.54mm:PinSocket_1x03_P2.54mm_Vertical, F.Cu at (29.5, 153.8)
- added JP2: 3V3 / 10V, Jumper:SolderJumper-3_P1.3mm_Open_RoundedPad1.0x1.5mm, F.Cu at (291.7, 20.8)
- added JP3: PIN / GND, Jumper:SolderJumper-3_P1.3mm_Bridged12_RoundedPad1.0x1.5mm, F.Cu at (253.5, 132.4)
- added JP4: CONN / BOARD, Jumper:SolderJumper-3_P1.3mm_Bridged12_RoundedPad1.0x1.5mm, F.Cu at (286.5, 49.7)
- added JP5: CONN / BOARD, Jumper:SolderJumper-3_P1.3mm_Bridged12_RoundedPad1.0x1.5mm, F.Cu at (286.5, 53.5)
- added JP6: CONN / BOARD, Jumper:SolderJumper-3_P1.3mm_Bridged12_RoundedPad1.0x1.5mm, F.Cu at (286.5, 57.4)
- added JP7: CONN / BOARD, Jumper:SolderJumper-3_P1.3mm_Bridged12_RoundedPad1.0x1.5mm, F.Cu at (286.5, 61.2)
- added L1: L, Inductor_SMD:L_Coilcraft_XAL7070-XXX, F.Cu at (50.0, 150.0)
- added L2: L, Inductor_SMD:L_Coilcraft_XAL7070-XXX, F.Cu at (125.0, 150.0)
- added L3: L, Inductor_SMD:L_Coilcraft_XAL7070-XXX, F.Cu at (87.5, 150.0)
- added L4: L_Ferrite, Inductor_SMD:L_0603_1608Metric, F.Cu at (261.3, 30.3)
- added R121: 2k20, Resistor_SMD:R_0402_1005Metric, F.Cu at (75.7, 159.5)
- added R122: 0, Resistor_SMD:R_0402_1005Metric, F.Cu at (83.5, 157.0)
- added R123: 2k20, Resistor_SMD:R_0402_1005Metric, F.Cu at (75.7, 160.5)
- added R124: 27k4, Resistor_SMD:R_0402_1005Metric, F.Cu at (91.5, 159.5)
- added R125: R_US, Resistor_SMD:R_0603_1608Metric, F.Cu at (38.8, 160.5)
- added R126: R_US, Resistor_SMD:R_0603_1608Metric, F.Cu at (38.8, 162.0)
- added R127: 2k20, Resistor_SMD:R_0402_1005Metric, F.Cu at (38.5, 157.5)
- added R128: 0, Resistor_SMD:R_0402_1005Metric, F.Cu at (46.0, 157.0)
- added R129: 2k20, Resistor_SMD:R_0402_1005Metric, F.Cu at (38.5, 156.5)
- added R130: 27k4, Resistor_SMD:R_0402_1005Metric, F.Cu at (54.0, 159.5)
- added R131: R_US, Resistor_SMD:R_0402_1005Metric, F.Cu at (113.2, 162.0)
- added R132: 10k, Resistor_SMD:R_0402_1005Metric, F.Cu at (166.5, 150.2)
- added R133: 10k, Resistor_SMD:R_0402_1005Metric, F.Cu at (166.0, 151.7)
- added R134: 10k, Resistor_SMD:R_0402_1005Metric, F.Cu at (164.5, 154.5)
- added R136: 10k, Resistor_SMD:R_0402_1005Metric, F.Cu at (163.3, 154.5)
- added R137: 10k, Resistor_SMD:R_0402_1005Metric, F.Cu at (162.0, 154.5)
- added R140: ?, Resistor_SMD:R_0603_1608Metric, F.Cu at (133.8, 29.0)
- added R141: ?, Resistor_SMD:R_0603_1608Metric, F.Cu at (133.8, 32.0)
- added R142: ?, Resistor_SMD:R_0603_1608Metric, F.Cu at (133.8, 35.0)
- added R143: ?, Resistor_SMD:R_0603_1608Metric, F.Cu at (133.8, 38.0)
- added R145: R_US, Resistor_SMD:R_0603_1608Metric, F.Cu at (31.8, 82.4)
- added R151: 0, Resistor_SMD:R_0402_1005Metric, F.Cu at (121.0, 157.0)
- added R152: R_US, Resistor_SMD:R_0603_1608Metric, F.Cu at (116.9, 195.7)
- added R158: R_US, Resistor_SMD:R_0603_1608Metric, F.Cu at (120.9, 185.7)
- added R159: 200k, Resistor_SMD:R_0402_1005Metric, F.Cu at (47.8, 187.0)
- added R162: 10m, Resistor_SMD:R_2512_6332Metric, F.Cu at (155.3, 149.0)
- added R164: 453k, Resistor_SMD:R_0603_1608Metric, F.Cu at (43.7, 173.9)
- added R165: 510, Resistor_SMD:R_0603_1608Metric, F.Cu at (43.7, 176.4)
- added R167: 33k2, Resistor_SMD:R_0603_1608Metric, F.Cu at (43.7, 179.0)
- added R168: 49k9, Resistor_SMD:R_0603_1608Metric, F.Cu at (43.7, 181.5)
- added R171: 1k, Resistor_SMD:R_0402_1005Metric, F.Cu at (195.8, 38.4)
- added R172: 1k, Resistor_SMD:R_0402_1005Metric, F.Cu at (195.8, 40.4)
- added R173: 0, Resistor_SMD:R_0603_1608Metric, F.Cu at (166.8, 38.7)
- added R174: 0, Resistor_SMD:R_0603_1608Metric, F.Cu at (166.8, 41.2)
- added R176: 60, Resistor_SMD:R_0603_1608Metric, F.Cu at (166.8, 43.7)
- added R177: 60, Resistor_SMD:R_0603_1608Metric, F.Cu at (166.8, 46.2)
- added R178: 1k, Resistor_SMD:R_0402_1005Metric, F.Cu at (195.8, 42.4)
- added R179: 1k, Resistor_SMD:R_0402_1005Metric, F.Cu at (195.8, 44.4)
- added R180: 0, Resistor_SMD:R_0201_0603Metric, F.Cu at (192.3, 52.8)
- added R181: 0, Resistor_SMD:R_0201_0603Metric, F.Cu at (302.6, 12.9)
- added R182: 5.1k, Resistor_SMD:R_0603_1608Metric, F.Cu at (166.8, 48.7)
- added R184: R_US, Resistor_SMD:R_0603_1608Metric, F.Cu at (166.8, 51.2)
- added R185: 10k, Resistor_SMD:R_0402_1005Metric, F.Cu at (312.5, 20.0)
- added R186: 10k, Resistor_SMD:R_0402_1005Metric, F.Cu at (312.5, 22.0)
- added R187: 10k, Resistor_SMD:R_0402_1005Metric, F.Cu at (312.5, 24.0)
- added R188: 10k, Resistor_SMD:R_0402_1005Metric, F.Cu at (312.5, 26.0)
- added R189: 10k, Resistor_SMD:R_0402_1005Metric, F.Cu at (312.5, 28.0)
- added R190: 10k, Resistor_SMD:R_0402_1005Metric, F.Cu at (312.5, 30.0)
- added R191: 10k, Resistor_SMD:R_0402_1005Metric, F.Cu at (312.5, 32.0)
- added R192: 10k, Resistor_SMD:R_0402_1005Metric, F.Cu at (315.4, 20.0)
- added R193: 10k, Resistor_SMD:R_0402_1005Metric, F.Cu at (315.4, 22.0)
- added R194: 10k, Resistor_SMD:R_0402_1005Metric, F.Cu at (315.4, 24.0)
- added R195: 10k, Resistor_SMD:R_0402_1005Metric, F.Cu at (315.4, 26.0)
- added R196: ?, Resistor_SMD:R_0603_1608Metric, F.Cu at (315.9, 39.2)
- added R197: 10k, Resistor_SMD:R_0402_1005Metric, F.Cu at (315.4, 28.0)
- added R198: 10k, Resistor_SMD:R_0402_1005Metric, F.Cu at (315.4, 30.0)
- added R199: 10k, Resistor_SMD:R_0402_1005Metric, F.Cu at (315.4, 32.0)
- added R200: 10k, Resistor_SMD:R_0402_1005Metric, F.Cu at (318.3, 20.0)
- added R201: 10k, Resistor_SMD:R_0402_1005Metric, F.Cu at (318.3, 22.0)
- added R202: 10k, Resistor_SMD:R_0402_1005Metric, F.Cu at (318.3, 24.0)
- added R203: 10k, Resistor_SMD:R_0402_1005Metric, F.Cu at (318.3, 26.0)
- added R204: 0, Resistor_SMD:R_0201_0603Metric, F.Cu at (256.2, 143.0)
- added R205: 1k, Resistor_SMD:R_0603_1608Metric, F.Cu at (251.9, 114.8)
- added R206: ?, Resistor_SMD:R_0603_1608Metric, F.Cu at (251.2, 139.4)
- added R207: 0, Resistor_SMD:R_0201_0603Metric, F.Cu at (256.2, 144.8)
- added R208: 1k, Resistor_SMD:R_0603_1608Metric, F.Cu at (251.9, 119.8)
- added R209: 0, Resistor_SMD:R_0201_0603Metric, F.Cu at (256.2, 146.5)
- added R210: 1k, Resistor_SMD:R_0603_1608Metric, F.Cu at (251.9, 122.3)
- added R211: 1k, Resistor_SMD:R_0603_1608Metric, F.Cu at (255.9, 112.3)
- added R212: 1k, Resistor_SMD:R_0603_1608Metric, F.Cu at (255.9, 114.8)
- added R213: 1k, Resistor_SMD:R_0603_1608Metric, F.Cu at (255.9, 117.3)
- added R214: 1k, Resistor_SMD:R_0402_1005Metric, F.Cu at (267.4, 107.5)
- added R215: 1k, Resistor_SMD:R_0402_1005Metric, F.Cu at (267.4, 109.5)
- added R216: ?, Resistor_SMD:R_0603_1608Metric, F.Cu at (281.7, 49.2)
- added R217: ?, Resistor_SMD:R_0603_1608Metric, F.Cu at (281.7, 51.7)
- added R218: 10k, Resistor_SMD:R_0603_1608Metric_Pad0.98x0.95mm_HandSolder, F.Cu at (291.5, 58.1)
- added R219: ?, Resistor_SMD:R_0603_1608Metric, F.Cu at (281.7, 54.2)
- added R220: 10k, Resistor_SMD:R_0603_1608Metric_Pad0.98x0.95mm_HandSolder, F.Cu at (291.5, 60.6)
- added R221: ?, Resistor_SMD:R_0603_1608Metric, F.Cu at (281.7, 56.7)
- added R222: ?, Resistor_SMD:R_0603_1608Metric, F.Cu at (281.7, 59.2)
- added R223: ?, Resistor_SMD:R_0603_1608Metric, F.Cu at (281.7, 61.7)
- added R224: 1k, Resistor_SMD:R_0603_1608Metric, F.Cu at (281.7, 64.2)
- added R225: 1k, Resistor_SMD:R_0603_1608Metric, F.Cu at (281.7, 66.7)
- added R226: 0, Resistor_SMD:R_0201_0603Metric, F.Cu at (276.3, 70.0)
- added R227: 0, Resistor_SMD:R_0201_0603Metric, F.Cu at (276.3, 71.8)
- added SW1: BOOT, Connector_PinSocket_2.54mm:PinSocket_1x03_P2.54mm_Vertical, F.Cu at (261.6, 43.8)
- added U10: ~, Package_BGA:LFBGA-153_11.5x13mm_Layout14x14_P0.5mm, F.Cu at (303.8, 27.1)
- added U4: TPS55285, Library:WQFN-HR - 15, F.Cu at (50.0, 158.5)
- added U5: LT3042xMSE, Package_SO:MSOP-10-1EP_3x3mm_P0.5mm_EP1.68x1.88mm, F.Cu at (128.4, 179.5)
- added U7: LT3042xMSE, Package_SO:MSOP-10-1EP_3x3mm_P0.5mm_EP1.68x1.88mm, F.Cu at (53.3, 180.2)
- added U9: USBLC6-2SC6, Package_TO_SOT_SMD:SOT-23-6, F.Cu at (180.0, 52.1)
- C1, C10, C11, C12, C13, C14, C15, C16, C17, C18, C19, C2, C20, C3, C4, C5, C6, C7, C8, C9: value 100nF -> 100n; footprint Capacitor_SMD:C_0603_1608Metric -> Capacitor_SMD:C_0402_1005Metric
- C23, C25, C26, C28, C29, C93: footprint Capacitor_SMD:C_0603_1608Metric -> Capacitor_SMD:C_0402_1005Metric
- C30: value 0.1uF -> 0u1
- C35, C52: value 0.1u -> C; footprint Capacitor_SMD:C_0603_1608Metric -> Capacitor_SMD:C_1206_3216Metric
- C36, C39: value ? -> C
- C37: value ? -> C; footprint Capacitor_SMD:C_0603_1608Metric -> Capacitor_SMD:C_1206_3216Metric
- C38: value DNF -> C
- C40, C56, C92: value 0.1u -> C; footprint Capacitor_SMD:C_0603_1608Metric -> Capacitor_SMD:C_0402_1005Metric
- C41: value 10u -> C; footprint Capacitor_SMD:C_0603_1608Metric -> Capacitor_SMD:C_0402_1005Metric
- C42, C43: value 10nF -> C; footprint Capacitor_SMD:C_0603_1608Metric -> Capacitor_SMD:C_1206_3216Metric
- C44: value 10nF -> C; footprint Capacitor_SMD:C_0603_1608Metric -> Capacitor_SMD:C_0402_1005Metric
- C46: value 100nF -> 100p; footprint Capacitor_SMD:C_0603_1608Metric -> Capacitor_SMD:C_0402_1005Metric
- C47: value 2.2u -> ?; footprint Capacitor_SMD:C_0603_1608Metric -> Capacitor_SMD:C_0402_1005Metric
- C48: value 0.1u -> C
- C49, C50, C54: value 0.1u -> 4u7; footprint Capacitor_SMD:C_0603_1608Metric -> Capacitor_SMD:C_1206_3216Metric
- C51: value 10u -> C; footprint Capacitor_SMD:C_0603_1608Metric -> Capacitor_SMD:C_1206_3216Metric
- C57: value C -> 100n; footprint Capacitor_SMD:C_0603_1608Metric -> Capacitor_SMD:C_0402_1005Metric
- C60: value CdV/dT -> DNF; footprint Capacitor_SMD:C_0603_1608Metric -> Capacitor_SMD:C_0402_1005Metric
- C61: value 0.1u -> DNF; footprint Capacitor_SMD:C_0603_1608Metric -> Capacitor_SMD:C_0402_1005Metric
- C62, C63, C64, C66, C75: value C -> 0u1; footprint Capacitor_SMD:C_0603_1608Metric -> Capacitor_SMD:C_0402_1005Metric
- C67: value 4.7u ESR < 100m -> 0u1; footprint Capacitor_SMD:C_0603_1608Metric -> Capacitor_SMD:C_0402_1005Metric
- C68, C69: value 2.2u ESR < 100m -> 0u1; footprint Capacitor_SMD:C_0603_1608Metric -> Capacitor_SMD:C_0402_1005Metric
- C70: value 4.7u -> 0u1; footprint Capacitor_SMD:C_0603_1608Metric -> Capacitor_SMD:C_0402_1005Metric
- C71: value 4.7u -> 10u
- C72: value 220p -> 2.2u
- C73, C74: value 10u ESR < 20m -> 0u1; footprint Capacitor_SMD:C_0603_1608Metric -> Capacitor_SMD:C_0402_1005Metric
- C76, C78, C82: value C -> ?; footprint Capacitor_SMD:C_0603_1608Metric -> Capacitor_SMD:C_0402_1005Metric
- C77: value C -> 10n; footprint Capacitor_SMD:C_0603_1608Metric -> Capacitor_SMD:C_0402_1005Metric
- C79, C80: value C -> 1u; footprint Capacitor_SMD:C_0603_1608Metric -> Capacitor_SMD:C_0402_1005Metric
- C81: value C -> DNF
- C83, C85: value C -> 10n
- C84: value C -> 10u
- C86: value 0.1u -> 220n
- C87: value 0.1u -> 10n
- C88: value 0.1u -> 2u2
- C89: value C -> 2u2
- C94: value C -> 100p; footprint Capacitor_SMD:C_0603_1608Metric -> Capacitor_SMD:C_0402_1005Metric
- D2: value 6.4V -> VBATT+; footprint Diode_SMD:D_0603_1608Metric_Pad1.05x0.95mm_HandSolder -> LED_SMD:LED_0603_1608Metric
- D4: value BAV99 -> VDD_3V3; footprint Package_TO_SOT_SMD:SOT-23 -> LED_SMD:LED_0603_1608Metric
- D5: value BAV99 -> VDDA_3V3; footprint Package_TO_SOT_SMD:SOT-23 -> LED_SMD:LED_0603_1608Metric
- J1: value JTAG -> PORT_G; footprint UserFootprints:490107670612 -> Connector_PinSocket_2.54mm:PinSocket_1x16_P2.54mm_Vertical
- J2: value USB_C_Receptacle_USB2.0_man -> PORT_E; footprint Connector_USB:USB_C_Receptacle_GCT_USB4105-xx-A_16P_TopMnt_Horizontal -> Connector_PinSocket_2.54mm:PinSocket_1x16_P2.54mm_Vertical
- J3: value Micro_SD_Card_Det1 -> PORT_F; footprint UserFootprints:GCT_MEM2075-00-140-01-A -> Connector_PinSocket_2.54mm:PinSocket_1x16_P2.54mm_Vertical
- R135: value 0 -> 10k; footprint Resistor_SMD:R_0201_0603Metric -> Resistor_SMD:R_0402_1005Metric
- R138, R139: value 0 -> R_US; footprint Resistor_SMD:R_0201_0603Metric -> Resistor_SMD:R_0603_1608Metric
- R14, R15: value 10k -> 0; footprint Resistor_SMD:R_0402_1005Metric -> Resistor_SMD:R_0201_0603Metric
- R144, R156: footprint Resistor_SMD:R_0402_1005Metric -> Resistor_SMD:R_0603_1608Metric
- R146, R150: value R_US -> 10m; footprint Resistor_SMD:R_0603_1608Metric -> Resistor_SMD:R_2512_6332Metric
- R147: footprint Resistor_SMD:R_0603_1608Metric -> Resistor_SMD:R_0402_1005Metric
- R148, R153: value R_US -> 2k20; footprint Resistor_SMD:R_0603_1608Metric -> Resistor_SMD:R_0402_1005Metric
- R149: value R_US -> 200k; footprint Resistor_SMD:R_0603_1608Metric -> Resistor_SMD:R_0402_1005Metric
- R155: value R_US -> 27k4
- R175: renamed from R13; value R_US -> 0
- R50: value DNF -> R_US
- R6: value ? -> R_US; footprint Resistor_SMD:R_0603_1608Metric -> Resistor_SMD:R_0402_1005Metric
- R7: value 0 -> R_US; footprint Resistor_SMD:R_0201_0603Metric -> Resistor_SMD:R_0402_1005Metric
- U11: value LT3042xMSE -> INA826; footprint Package_SO:MSOP-10-1EP_3x3mm_P0.5mm_EP1.68x1.88mm -> Package_SO:SOIC-8-1EP_3.9x4.9mm_P1.27mm_EP2.29x3mm
- U2: value ~ -> INA3221; footprint Package_BGA:LFBGA-153_11.5x13mm_Layout14x14_P0.5mm -> Package_DFN_QFN:Texas_RGV0016A_VQFN-16-1EP_4x4mm_P0.65mm_EP2.1x2.1mm
- U3: value INA826 -> TPS55285; footprint UserFootprints:SOP65P490X110-8N -> Library:WQFN-HR - 15
- U6: value INA219AxD -> TPS55285; footprint Package_SO:SOIC-8_3.9x4.9mm_P1.27mm -> Library:WQFN-HR - 15
- U8: value INA219AxD -> TCAN337G
- moved C68 253.0 mm to (312.5, 35.9)
- moved C67 252.8 mm to (312.5, 33.9)
- moved C71 247.0 mm to (315.9, 34.2)
- moved C72 247.0 mm to (315.9, 36.7)
- moved C74 243.0 mm to (312.5, 43.8)
- moved C73 242.8 mm to (312.5, 41.8)
- moved C70 240.7 mm to (312.5, 39.9)
- moved C69 240.5 mm to (312.5, 37.9)
- moved C66 239.7 mm to (286.3, 13.1)
- moved C62 233.8 mm to (283.4, 13.1)
- moved C84 214.5 mm to (270.7, 37.5)
- moved C89 210.7 mm to (261.3, 25.3)
- moved C29 202.7 mm to (260.7, 40.4)
- moved C28 202.4 mm to (260.7, 38.5)
- moved C26 202.1 mm to (260.7, 36.5)
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- renumbered R96 to R10, R193 to R100, R162 to R101, R194 to R102, R163 to R103, R195 to R104, R164 to R105, R165 to R106, R166 to R107, R167 to R108, R168 to R109, R199 to R11, R169 to R110, R170 to R111, R171 to R112, R172 to R113, R173 to R114, R174 to R115, R175 to R116, R176 to R117, R177 to R118, R178 to R119, R103 to R12, R179 to R120, R200 to R13, R104 to R16, R201 to R17, R105 to R18, R4 to R183, R202 to R19, R79 to R2, R106 to R20, R203 to R21, R107 to R22, R204 to R23, R108 to R24, R205 to R25, R109 to R26, R206 to R27, R110 to R28, R207 to R29, R196 to R3, R111 to R30, R208 to R31, R112 to R32, R209 to R33, R113 to R34, R210 to R35, R114 to R36, R211 to R37, R115 to R38, R212 to R39, R80 to R4, R116 to R40, R213 to R41, R117 to R42, R214 to R43, R118 to R44, R215 to R45, R119 to R46, R216 to R47, R120 to R48, R217 to R49, R197 to R5, R121 to R51, R218 to R52, R122 to R53, R219 to R54, R131 to R55, R123 to R56, R220 to R57, R132 to R58, R124 to R59, R221 to R60, R125 to R61, R222 to R62, R126 to R63, R223 to R64, R127 to R65, R224 to R66, R128 to R67, R225 to R68, R129 to R69, R226 to R70, R130 to R71, R227 to R72, R133 to R73, R180 to R74, R134 to R75, R181 to R76, R136 to R77, R182 to R78, R137 to R79, R95 to R8, R183 to R80, R141 to R81, R184 to R82, R142 to R83, R185 to R84, R143 to R85, R186 to R86, R151 to R87, R187 to R88, R152 to R89, R198 to R9, R188 to R90, R157 to R91, R189 to R92, R158 to R93, R190 to R94, R159 to R95, R191 to R96, R160 to R97, R192 to R98, R161 to R99, U7 to U1
Connections:
- C23 pad 1: VREF+ -> VDDA_MCU
- C25 pad 1: VDDA_MCU -> VREF+
- C30 pad 1: VBUS -> VDD_3V3
- C35 pad 1: GND -> VBAT_SAFE
- C35 pad 2: VDDA -> GND
- C36 pad 1: Net-(U3--) -> /POWER/TPS3V3_VCC
- C37 pad 1: Net-(U3-+) -> /POWER/TPS10V_VIN
- C37 pad 2: Net-(U3--) -> GND
- C38 pad 1: GND -> /POWER/TPS10V_VIN
- C38 pad 2: /ADC/PT1 -> GND
- C39 pad 1: GND -> /POWER/TPS10V_VCC
- C39 pad 2: Net-(U3-+) -> GND
- C40 pad 1: GND -> Net-(U4-EN/UVLO)
- C40 pad 2: VDD_3V3 -> GND
- C41 pad 1: GND -> /POWER/L1_L
- C41 pad 2: VDD_3V3 -> Net-(U4-BOOT1)
- C42 pad 1: /ADC/-IN3 -> /POWER/TPS3V3A_VOUT
- C42 pad 2: /ADC/+IN3 -> GND
- C43 pad 1: /ADC/-IN4 -> /POWER/Psense2_IN+
- C43 pad 2: /ADC/+IN4 -> GND
- C44 pad 1: /ADC/-IN5 -> /POWER/L1_R
- C44 pad 2: /ADC/+IN5 -> Net-(U4-BOOT2)
- C46 pad 1: VDD_3V3 -> Net-(U4-COMP)
- C47 pad 1: VDD_3V3 -> Net-(C47-Pad1)
- C48 pad 1: VDD_3V3 -> /POWER/TPS10V_VOUT
- C49 pad 1: VDD_3V3 -> /POWER/TPS10V_VOUT
- C50 pad 1: VDD_3V3 -> /POWER/Psense3_IN+
- C51 pad 1: VDD_3V3 -> /POWER/TPS10V_VOUT
- C52 pad 1: VDD_3V3 -> VBAT_SAFE
- C53 pad 1: Net-(U6-IN-) -> VBAT_SAFE
- C53 pad 2: Net-(U6-IN+) -> GND
- C54 pad 1: GND -> Net-(U7-SET)
- C54 pad 2: VDD_3V3 -> GND
- C55 pad 1: Net-(U8-IN-) -> /POWER/TPS3V3A_VCC
- C55 pad 2: Net-(U8-IN+) -> GND
- C56 pad 1: GND -> Net-(U6-EN/UVLO)
- C56 pad 2: VDD_3V3 -> GND
- C57 pad 1: Net-(U13-IN-) -> GND
- C57 pad 2: Net-(U13-IN+) -> VDD_3V3
- C60 pad 1: Net-(IC1-DVDT) -> GND
- C60 pad 2: GND -> /COMMUNICATION/CANH
- C61 pad 2: VDD_3V3 -> /COMMUNICATION/CANL
- C62 pad 1: Net-(JP13-C) -> GND
- C62 pad 2: GND -> Net-(C62-Pad2)
- C63 pad 1: Net-(U9-SW1) -> GND
- C64 pad 1: Net-(U9-SW2) -> VDD50_USB
- C64 pad 2: Net-(U9-BOOT2) -> GND
- C66 pad 1: Net-(U9-COMP) -> GND
- C66 pad 2: GND -> Net-(J16-SHIELD)
- C67 pad 1: VDDSMPS -> VDD_3V3
- C68 pad 1: Net-(JP8-A) -> VDD_3V3
- C69 pad 1: Net-(JP9-A) -> VDD_3V3
- C70 pad 1: Net-(JP10-A) -> VDD_3V3
- C71 pad 1: Net-(JP11-A) -> VDD_3V3
- C72 pad 1: /VLXSMPS -> VDD_3V3
- C73 pad 1: /VFBSMPS -> Net-(J17-SHIELD)
- C74 pad 1: Net-(JP12-A) -> GND
- C74 pad 2: GND -> VDD_3V3
- C75 pad 1: Net-(C75-Pad1) -> GND
- C75 pad 2: GND -> VDDA
- C76 pad 1: Net-(U14-EN/UV) -> Net-(U11-+)
- C77 pad 1: Net-(U14-SET) -> /ADC/-IN2
- C77 pad 2: GND -> /ADC/+IN2
- C78 pad 1: /POWER/Psense3_IN+ -> Net-(U11--)
- C78 pad 2: GND -> Net-(U11-+)
- C79 pad 1: Net-(U10-SW1) -> GND
- C79 pad 2: Net-(U10-BOOT1) -> VDDA_3V3
- C80 pad 1: Net-(U10-SW2) -> VDD_3V3
- C80 pad 2: Net-(U10-BOOT2) -> GND
- C81 pad 1: VBAT_SAFE -> GND
- C81 pad 2: GND -> /ADC/PT1
- C82 pad 1: Net-(U10-VCC) -> GND
- C82 pad 2: GND -> Net-(U11--)
- C83 pad 1: 3V5 -> /ADC/-IN3
- C83 pad 2: GND -> /ADC/+IN3
- C84 pad 1: Net-(U10-COMP) -> GND
- C84 pad 2: GND -> VDDA
- C85 pad 1: Net-(C85-Pad1) -> /ADC/-IN4
- C85 pad 2: GND -> /ADC/+IN4
- C86 pad 2: Net-(J2-SHIELD) -> Net-(U12-CAP)
- C87 pad 1: GND -> /ADC/-IN5
- C87 pad 2: Net-(J8-PAD) -> /ADC/+IN5
- C88 pad 1: GND -> VCAP
- C88 pad 2: Net-(C88-Pad2) -> GND
- C89 pad 1: 3V5 -> VCAP
- C92 pad 1: Net-(J3-SHIELD) -> /POWER/L3_L
- C92 pad 2: GND -> Net-(U3-BOOT1)
- C93 pad 1: /POWER/Psense2_IN+ -> /POWER/L3_R
- C93 pad 2: GND -> Net-(U3-BOOT2)
- C94 pad 1: Net-(U11-SET) -> Net-(U3-COMP)
- D2 pad 2: GND -> +BATT1
- D4 pad 1: GND -> Net-(D4-K)
- D5 pad 1: GND -> Net-(D5-K)
- D5 pad 2: VDD_3V3 -> VDDA_3V3
- J1 pad 1: VDD_3V3 -> Net-(J1-Pin_1)
- J1 pad 2: /COMMUNICATION/NRST -> Net-(J1-Pin_2)
- J1 pad 3: GND -> Net-(J1-Pin_3)
- J1 pad 4: /COMMUNICATION/SWO -> Net-(J1-Pin_4)
- J1 pad 5: /COMMUNICATION/SWCLK -> Net-(J1-Pin_5)
- J1 pad 6: /COMMUNICATION/SWDIO -> Net-(J1-Pin_6)
- J3 pad 1: /STORAGE/SD_DAT2 -> Net-(J3-Pin_1)
- J3 pad 10: Net-(J3-SHIELD) -> Net-(J3-Pin_10)
- J3 pad 2: /STORAGE/SD_DAT3 -> Net-(J3-Pin_2)
- J3 pad 3: /STORAGE/SD_CMD -> Net-(J3-Pin_3)
- J3 pad 4: VDD_3V3 -> Net-(J3-Pin_4)
- J3 pad 5: /STORAGE/SD_CLK -> Net-(J3-Pin_5)
- J3 pad 6: GND -> Net-(J3-Pin_6)
- J3 pad 7: /STORAGE/SD_DAT0 -> Net-(J3-Pin_7)
- J3 pad 8: /STORAGE/SD_DAT1 -> Net-(J3-Pin_8)
- J3 pad 9: /STORAGE/SD_DET -> Net-(J3-Pin_9)
- R1 pad 1: VDD_10V -> VDDA_3V3
- R1 pad 2: VDDA -> VREF+
- R10 pad 1: Net-(J14-Pin_4) -> Net-(J1-Pin_4)
- R11 pad 2: Net-(J16-Pin_4) -> Net-(J2-Pin_4)
- R12 pad 1: Net-(J14-Pin_5) -> Net-(J1-Pin_5)
- R13 pad 2: Net-(J16-Pin_5) -> Net-(J2-Pin_5)
- R135 pad 1: /OTG_USB -> VDD_3V3
- R135 pad 2: VBUS -> /POWER/PM_TC
- R138 pad 1: VDD33_USB -> Net-(D6-K)
- R138 pad 2: VDD50_USB -> Net-(IC1-~{EN}/OVLO)
- R139 pad 1: VDD_MCU -> /POWER/EFUSE_FLT
- R14 pad 1: VDD_3V3 -> VDD_MCU
- R14 pad 2: /STORAGE/eMMC_DAT7 -> VDD_3V3
- R144 pad 1: VDD_MCU -> Net-(IC1-~{EN}/OVLO)
- R144 pad 2: /NRST -> GND
- R146 pad 1: /POWER/Psense2_IN+ -> /POWER/Psense1_IN+
- R146 pad 2: Net-(U11-PGFB) -> VDD_3V3
- R147 pad 1: Net-(U11-ILIM) -> Net-(U6-EN/UVLO)
- R148 pad 1: Net-(U11-SET) -> VDD_3V3
- R148 pad 2: GND -> /POWER/TPS3V3A_SCL
- R149 pad 1: Net-(U11-PGFB) -> /POWER/TPS3V3A_VOUT
- R149 pad 2: GND -> Net-(U5-PG)
- R15 pad 2: /STORAGE/eMMC_DAT6 -> VDDA_MCU
- R150 pad 1: GND -> /POWER/Psense2_IN+
- R150 pad 2: Net-(Q6-E) -> VDDA_3V3
- R153 pad 1: GND -> VDD_3V3
- R153 pad 2: Net-(Q5-E) -> /POWER/TPS3V3A_SDA
- R154 pad 1: GND -> Net-(U5-ILIM)
- R154 pad 2: Net-(Q3-E) -> GND
- R155 pad 1: VDD_3V3 -> Net-(U6-COMP)
- R155 pad 2: /COMMUNICATION/ADXL_SDA -> Net-(C104-Pad1)
- R156 pad 1: VDD_3V3 -> Net-(U5-SET)
- R156 pad 2: /COMMUNICATION/ADXL_SCL -> GND
- R16 pad 1: Net-(J14-Pin_6) -> Net-(J1-Pin_6)
- R17 pad 2: Net-(J16-Pin_6) -> Net-(J2-Pin_6)
- R175 pad 2: GND -> VDD_3V3
- R18 pad 1: Net-(J14-Pin_7) -> Net-(J1-Pin_7)
- R183 pad 1: Net-(J2-CC2) -> Net-(J16-CC2)
- R19 pad 2: Net-(J16-Pin_7) -> Net-(J2-Pin_7)
- R2 pad 1: Net-(J14-Pin_1) -> Net-(J1-Pin_1)
- R20 pad 1: Net-(J14-Pin_8) -> Net-(J1-Pin_8)
- R21 pad 2: Net-(J16-Pin_8) -> Net-(J2-Pin_8)
- R22 pad 1: Net-(J14-Pin_9) -> Net-(J1-Pin_9)
- R23 pad 2: Net-(J16-Pin_9) -> Net-(J2-Pin_9)
- R24 pad 1: Net-(J14-Pin_10) -> Net-(J1-Pin_10)
- R25 pad 2: Net-(J16-Pin_10) -> Net-(J2-Pin_10)
- R26 pad 1: Net-(J14-Pin_11) -> Net-(J1-Pin_11)
- R27 pad 2: Net-(J16-Pin_11) -> Net-(J2-Pin_11)
- R28 pad 1: Net-(J14-Pin_12) -> Net-(J1-Pin_12)
- R29 pad 2: Net-(J16-Pin_12) -> Net-(J2-Pin_12)
- R3 pad 2: Net-(J16-Pin_1) -> Net-(J2-Pin_1)
- R30 pad 1: Net-(J14-Pin_13) -> Net-(J1-Pin_13)
- R31 pad 2: Net-(J16-Pin_13) -> Net-(J2-Pin_13)
- R32 pad 1: Net-(J14-Pin_14) -> Net-(J1-Pin_14)
- R33 pad 2: Net-(J16-Pin_14) -> Net-(J2-Pin_14)
- R34 pad 1: Net-(J14-Pin_15) -> Net-(J1-Pin_15)
- R35 pad 2: Net-(J16-Pin_15) -> Net-(J2-Pin_15)
- R36 pad 1: Net-(J14-Pin_16) -> Net-(J1-Pin_16)
- R37 pad 2: Net-(J16-Pin_16) -> Net-(J2-Pin_16)
- R38 pad 1: Net-(J15-Pin_1) -> Net-(J3-Pin_1)
- R4 pad 1: Net-(J14-Pin_2) -> Net-(J1-Pin_2)
- R40 pad 1: Net-(J15-Pin_2) -> Net-(J3-Pin_2)
- R42 pad 1: Net-(J15-Pin_3) -> Net-(J3-Pin_3)
- R44 pad 1: Net-(J15-Pin_4) -> Net-(J3-Pin_4)
- R46 pad 1: Net-(J15-Pin_5) -> Net-(J3-Pin_5)
- R48 pad 1: Net-(J15-Pin_6) -> Net-(J3-Pin_6)
- R5 pad 2: Net-(J16-Pin_2) -> Net-(J2-Pin_2)
- R50 pad 1: VDD_3V3 -> VDD_MCU
- R50 pad 2: /STORAGE/SD_DAT1 -> /NRST
- R51 pad 1: Net-(J15-Pin_7) -> Net-(J3-Pin_7)
- R53 pad 1: Net-(J15-Pin_8) -> Net-(J3-Pin_8)
- R56 pad 1: Net-(J15-Pin_9) -> Net-(J3-Pin_9)
- R59 pad 1: Net-(J15-Pin_10) -> Net-(J3-Pin_10)
- R6 pad 1: Net-(R6-Pad1) -> VBAT_SAFE
- R6 pad 2: /ADC/INA1_RG- -> Net-(U3-EN/UVLO)
- R61 pad 1: Net-(J15-Pin_11) -> Net-(J3-Pin_11)
- R63 pad 1: Net-(J15-Pin_12) -> Net-(J3-Pin_12)
- R65 pad 1: Net-(J15-Pin_13) -> Net-(J3-Pin_13)
- R67 pad 1: Net-(J15-Pin_14) -> Net-(J3-Pin_14)
- R69 pad 1: Net-(J15-Pin_15) -> Net-(J3-Pin_15)
- R7 pad 1: /ADC/PT1 -> Net-(U3-EN/UVLO)
- R7 pad 2: Net-(U3-Vout) -> GND
- R71 pad 1: Net-(J15-Pin_16) -> Net-(J3-Pin_16)
- R8 pad 1: Net-(J14-Pin_3) -> Net-(J1-Pin_3)
- R9 pad 2: Net-(J16-Pin_3) -> Net-(J2-Pin_3)
- U1 pad 135: VDDLDO -> VDD_MCU
- U1 pad 15: /VLXSMPS -> unconnected-(U1A-VLXSMPS-Pad15)
- U1 pad 16: VDDSMPS -> VDD_MCU
- U1 pad 17: /VFBSMPS -> unconnected-(U1B-VFBSMPS-Pad17)
- U1 pad 175: VDDLDO -> VDD_MCU
- U1 pad 82: VDDLDO -> VDD_MCU
- U11 pad 1: 3V5 -> Net-(U11--)
- U11 pad 2: 3V5 -> Net-(U11-RG+)
- U11 pad 3: 3V5 -> Net-(U11-RG-)
- U11 pad 4: Net-(U11-PG) -> Net-(U11-+)
- U11 pad 5: Net-(U11-ILIM) -> GND
- U11 pad 6: Net-(U11-PGFB) -> Net-(JP3-C)
- U11 pad 7: Net-(U11-SET) -> Net-(U11-VOUT)
- U11 pad 8: GND -> VDDA
- U11 pad 9: /POWER/Psense2_IN+ -> (no net)
- U12 pad 1: VDDA -> VDDA_3V3
- U12 pad 18: unconnected-(U12-CAP-Pad18) -> Net-(U12-CAP)
- U12 pad 20: unconnected-(U12-DVDD-Pad20) -> VDD_3V3
- U3 pad 1: Net-(U3--) -> Net-(U3-MODE)
- U3 pad 2: /ADC/INA1_RG- -> /POWER/TPS3V3_SCL
- U3 pad 3: Net-(R6-Pad1) -> /POWER/TPS3V3_SDA
- U3 pad 4: Net-(U3-+) -> Net-(U3-EN/UVLO)
- U3 pad 5: GND -> VBAT_SAFE
- U3 pad 6: Net-(JP3-C) -> /POWER/L3_L
- U3 pad 7: Net-(U3-Vout) -> GND
- U3 pad 8: VDDA -> /POWER/L3_R
- U6 pad 1: GND -> Net-(U6-MODE)
- U6 pad 2: GND -> /POWER/TPS3V3A_SCL
- U6 pad 3: Net-(U6-SDA) -> /POWER/TPS3V3A_SDA
- U6 pad 4: Net-(U6-SCL) -> Net-(U6-EN/UVLO)
- U6 pad 5: VDD_3V3 -> VBAT_SAFE
- U6 pad 6: GND -> /POWER/L2_L
- U6 pad 7: Net-(U6-IN-) -> GND
- U6 pad 8: Net-(U6-IN+) -> /POWER/L2_R
- U8 pad 1: GND -> Net-(U8-TXD)
- U8 pad 2: VDD_3V3 -> GND
- U8 pad 3: Net-(U8-SDA) -> VDD_3V3
- U8 pad 5: VDD_3V3 -> /COMMUNICATION/TCAN_FLT
- U8 pad 6: GND -> /COMMUNICATION/CANL
- U8 pad 7: Net-(U8-IN-) -> /COMMUNICATION/CANH
- U8 pad 8: Net-(U8-IN+) -> /COMMUNICATION/TCAN_STBY
Routing:
- net VDD_3V3: track 0.00 -> 15.3 mm
- net Net-(U2-VPU): track 0.00 -> 9.97 mm, vias 0 -> 2
- net VDD_10V: track 0.00 -> 6.77 mm
- net /POWER/Psense1_IN+: track 0.00 -> 6.77 mm
- net VDDA_3V3: track 0.00 -> 6.73 mm
- net /POWER/Psense2_IN+: track 0.00 -> 6.73 mm
- net /POWER/Psense3_IN+: track 0.00 -> 6.69 mm
- net Net-(U6-COMP): track 0.00 -> 4.59 mm
- net Net-(U4-COMP): track 0.00 -> 4.59 mm
- net Net-(U3-COMP): track 0.00 -> 4.59 mm
- net Net-(U3-BOOT2): track 0.00 -> 2.94 mm
- net Net-(U3-BOOT1): track 0.00 -> 2.94 mm
- net Net-(U6-BOOT1): track 0.00 -> 2.94 mm
- net Net-(U4-BOOT2): track 0.00 -> 2.94 mm
- net Net-(U4-BOOT1): track 0.00 -> 2.94 mm
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- added copper zone on F.Cu, net /POWER/L1_L
- added copper zone on F.Cu, net /POWER/L1_R
- added copper zone on F.Cu, net /POWER/L2_L
- added copper zone on F.Cu, net /POWER/L2_R
- added copper zone on F.Cu, net /POWER/L3_L
- added copper zone on F.Cu, net /POWER/L3_R
- added copper zone on F.Cu, net /POWER/Psense1_IN+
- added copper zone on F.Cu, net /POWER/TPS10V_VCC
- added copper zone on F.Cu, net /POWER/TPS10V_VIN
- added copper zone on F.Cu, net /POWER/TPS10V_VOUT
- added copper zone on F.Cu, net /POWER/TPS3V3A_VCC
- added copper zone on F.Cu, net /POWER/TPS3V3A_VOUT
- added copper zone on F.Cu, net /POWER/TPS3V3_VCC
- added copper zone on F.Cu, net GND
- added copper zone on F.Cu, net VBAT_SAFE
