File: engine-control-unit_prototype/adc.kicad_sch (KiCad schematic)
At the start: 43 parts, among them J18 VREF, J19 PT1, J20 PT2, J21 PT3, J22 PT4, J23 PT5, U11 INA826, U12 ADS131M04xPW, Y4 SIT8924BA-22-33E-8.192000

Commit message: ajout de page root
Parts:
- removed C75: 0u1, Capacitor_SMD:C_0603_1608Metric, symbol Device:C
- removed C76, C78, C82: ?, Capacitor_SMD:C_0603_1608Metric, symbol Device:C
- removed C81: DNF, Capacitor_SMD:C_0402_1005Metric, symbol Device:C
- removed C84: 10u, Capacitor_SMD:C_0603_1608Metric, symbol Device:C
- removed J18: VREF, Connector_PinHeader_1.00mm:PinHeader_1x01_P1.00mm_Vertical, symbol Connector:Conn_01x01_Pin
- removed J19: PT1, Connector_PinSocket_2.54mm:PinSocket_1x04_P2.54mm_Vertical, symbol Connector:Screw_Terminal_01x04
- removed JP2: 3V3 / 10V, Jumper:SolderJumper-3_P1.3mm_Open_RoundedPad1.0x1.5mm, symbol Jumper:SolderJumper_3_Open
- removed JP3: PIN / GND, Jumper:SolderJumper-3_P1.3mm_Bridged12_RoundedPad1.0x1.5mm, symbol Jumper:SolderJumper_3_Bridged12
- removed R204, R209: 0, Resistor_SMD:R_0603_1608Metric, symbol Device:R_US
- removed R206: ?, Resistor_SMD:R_0402_1005Metric, symbol Device:R_US
- removed R207: 0, Resistor_SMD:R_0402_1005Metric, symbol Device:R_US
- removed U11: INA826, Package_SO:SOIC-8-1EP_3.9x4.9mm_P1.27mm_EP2.29x3mm, symbol SiriusLib:INA826
- renumbered C83 to C59, C85 to C60, C87 to C61, C77 to C62, C79 to C63, C80 to C64, C86 to C65, C129 to C66, C128 to C67, J23 to J10, J20 to J7, J21 to J8, J22 to J9, JP1 to JP2, R210 to R81, R211 to R82, R212 to R83, R213 to R84, R214 to R85, R215 to R86, R205 to R87, R208 to R88, R231 to R89, R172 to R90, R229 to R91, R230 to R92, U12 to U11, Y4 to Y1
Other:
- note added: "pull down"
- note removed: "(1)"
- note removed: "(2)"
- note removed: "(3)"
- note removed: "(4)"
- note removed: "(5)"
- note removed: "C0G ?"
