File: engine-control-unit_prototype/communication.kicad_sch (KiCad schematic)
At the start: 37 parts, among them J11 CANFD, J12 ADXL345, J13 MAG_CONN_1, J14 MAG_CONN_2, J15 JTAG, J16 USB_C_Receptacle_USB2.0_man, U14 TPS2069CDBV, U8 TCAN337G, U9 USBLC6-2SC6

Commit message: ajout de page root
Parts:
- J15: value JTAG -> SWD
Changed lines of the file:
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@@
 			)
 		)
-		(property "Value" "JTAG"
+		(property "Value" "SWD"
 			(at 213.36 144.78 0)
 			(effects
