File: engine-control-unit_prototype/storage.kicad_sch (KiCad schematic)
At the start: 29 parts, among them J3 Micro_SD_Card_Det1

Commit message: Added Control page Revisited power tree (VDDA_3V3 and VDD_3V3) Bunch of other fixes
Parts:
- C47, C48, C49, C50, C51, C52, C61, C92: footprint (none) -> Capacitor_SMD:C_0603_1608Metric
- R14, R15, R16, R17, R18, R19, R20, R21, R24, R32, R33: footprint (none) -> Resistor_SMD:R_0402_1005Metric
- R49, R50, R51, R52, R53, R54, R62: value DNF -> 10k; footprint (none) -> Resistor_SMD:R_0402_1005Metric
Changed lines of the file:
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@@
 			)
 		)
-		(property "Footprint" ""
+		(property "Footprint" "Capacitor_SMD:C_0603_1608Metric"
 			(at 214.9348 92.71 0)
 			(effects
@@
 			)
 		)
-		(property "Footprint" ""
+		(property "Footprint" "Resistor_SMD:R_0402_1005Metric"
 			(at 130.556 51.054 90)
 			(effects
@@
 			)
 		)
-		(property "Footprint" ""
+		(property "Footprint" "Capacitor_SMD:C_0603_1608Metric"
 			(at 272.0848 63.5 0)
 			(effects
@@
 			)
 		)
-		(property "Footprint" ""
+		(property "Footprint" "Resistor_SMD:R_0402_1005Metric"
 			(at 120.396 51.054 90)
 			(effects
@@
 			)
 		)
-		(property "Footprint" ""
+		(property "Footprint" "Resistor_SMD:R_0402_1005Metric"
 			(at 140.716 51.054 90)
 			(effects
@@
 			)
 		)
-		(property "Footprint" ""
+		(property "Footprint" "Capacitor_SMD:C_0603_1608Metric"
 			(at 221.2848 63.5 0)
 			(effects
@@
 			)
 		)
-		(property "Footprint" ""
+		(property "Footprint" "Capacitor_SMD:C_0603_1608Metric"
 			(at 83.82 171.1452 0)
 			(effects
@@
 			)
 		)
-		(property "Footprint" ""
+		(property "Footprint" "Resistor_SMD:R_0402_1005Metric"
 			(at 100.076 51.054 90)
 			(effects
@@
 			)
 		)
-		(property "Footprint" ""
+		(property "Footprint" "Resistor_SMD:R_0402_1005Metric"
 			(at 39.116 51.054 90)
 			(effects
@@
 			)
 		)
-		(property "Value" "DNF"
+		(property "Value" "10k"
 			(at 40.64 132.0799 0)
 			(effects
@@
 			)
 		)
-		(property "Footprint" ""
+		(property "Footprint" "Resistor_SMD:R_0402_1005Metric"
 			(at 42.164 131.064 90)
 			(effects
@@
 			)
 		)
-		(property "Footprint" ""
+		(property "Footprint" "Capacitor_SMD:C_0603_1608Metric"
 			(at 246.6848 63.5 0)
 			(effects
@@
 			)
 		)
-		(property "Footprint" ""
+		(property "Footprint" "Resistor_SMD:R_0402_1005Metric"
 			(at 59.436 51.054 90)
 			(effects
@@
 			)
 		)
-		(property "Value" "DNF"
+		(property "Value" "10k"
 			(at 60.96 132.0799 0)
 			(effects
@@
 			)
 		)
-		(property "Footprint" ""
+		(property "Footprint" "Resistor_SMD:R_0402_1005Metric"
 			(at 62.484 131.064 90)
 			(effects
@@
 			)
 		)
-		(property "Footprint" ""
+		(property "Footprint" "Resistor_SMD:R_0402_1005Metric"
 			(at 79.756 51.054 90)
 			(effects
@@
 			)
 		)
-		(property "Footprint" ""
+		(property "Footprint" "Resistor_SMD:R_0402_1005Metric"
 			(at 69.596 51.054 90)
 			(effects
@@
 			)
 		)
-		(property "Value" "DNF"
+		(property "Value" "10k"
 			(at 81.28 132.0799 0)
 			(effects
@@
 			)
 		)
-		(property "Footprint" ""
+		(property "Footprint" "Resistor_SMD:R_0402_1005Metric"
 			(at 82.804 131.064 90)
 			(effects
@@
 			)
 		)
-		(property "Footprint" ""
+		(property "Footprint" "Resistor_SMD:R_0402_1005Metric"
 			(at 49.276 51.054 90)
 			(effects
@@
 			)
 		)
-		(property "Footprint" ""
+		(property "Footprint" "Capacitor_SMD:C_0603_1608Metric"
 			(at 259.3848 63.5 0)
 			(effects
@@
 			)
 		)
-		(property "Footprint" ""
+		(property "Footprint" "Resistor_SMD:R_0402_1005Metric"
 			(at 89.916 51.054 90)
 			(effects
@@
 			)
 		)
-		(property "Value" "DNF"
+		(property "Value" "10k"
 			(at 50.8 132.0799 0)
 			(effects
@@
 			)
 		)
-		(property "Footprint" ""
+		(property "Footprint" "Resistor_SMD:R_0402_1005Metric"
 			(at 52.324 131.064 90)
 			(effects
@@
 			)
 		)
-		(property "Footprint" ""
+		(property "Footprint" "Resistor_SMD:R_0402_1005Metric"
 			(at 110.236 51.054 90)
 			(effects
@@
 			)
 		)
-		(property "Footprint" ""
+		(property "Footprint" "Capacitor_SMD:C_0603_1608Metric"
 			(at 233.9848 63.5 0)
 			(effects
@@
 		(property "Digikey" "https://www.digikey.ca/en/products/detail/alliance-memory-inc/ASFC32G31T3-51BIN/21801876"
 			(at 194.31 66.04 0)
+			(effects
+				(font
+					(size 1.27 1.27)
+				)
+				(hide yes)
+			)
+		)
+		(property "Link" ""
+			(at 194.31 68.58 0)
+			(effects
+				(font
+					(size 1.27 1.27)
+				)
+				(hide yes)
+			)
+		)
+		(property "Part Number" ""
+			(at 194.31 68.58 0)
 			(effects
 				(font
@@
 			)
 		)
+		(property "Link" ""
+			(at 157.48 72.39 0)
+			(effects
+				(font
+					(size 1.27 1.27)
+				)
+				(hide yes)
+			)
+		)
+		(property "Part Number" ""
+			(at 157.48 72.39 0)
+			(effects
+				(font
+					(size 1.27 1.27)
+				)
+				(hide yes)
+			)
+		)
 		(pin "C2"
 		)
@@
 			)
 		)
-		(property "Value" "DNF"
+		(property "Value" "10k"
 			(at 91.44 132.0799 0)
 			(effects
@@
 			)
 		)
-		(property "Footprint" ""
+		(property "Footprint" "Resistor_SMD:R_0402_1005Metric"
 			(at 92.964 131.064 90)
 			(effects
@@
 			)
 		)
-		(property "Value" "DNF"
+		(property "Value" "10k"
 			(at 30.48 132.0799 0)
 			(effects
@@
 			)
 		)
-		(property "Footprint" ""
+		(property "Footprint" "Resistor_SMD:R_0402_1005Metric"
 			(at 32.004 131.064 90)
 			(effects
@@
 			)
 		)
-		(property "Value" "DNF"
+		(property "Value" "10k"
 			(at 71.12 132.0799 0)
 			(effects
@@
 			)
 		)
-		(property "Footprint" ""
+		(property "Footprint" "Resistor_SMD:R_0402_1005Metric"
 			(at 72.644 131.064 90)
 			(effects
@@
 			)
 		)
-		(property "Footprint" ""
+		(property "Footprint" "Capacitor_SMD:C_0603_1608Metric"
 			(at 143.2052 168.91 0)
 			(effects

Commit message: Added magnetic encoders Added optional external valve control connector
Parts:
- renumbered C48 to C67, C50 to C68, C49 to C69, C52 to C70, C51 to C71, C47 to C72, C92 to C73, C61 to C74, J3 to J17, R32 to R185, R24 to R186, R21 to R187, R20 to R188, R19 to R189, R18 to R190, R17 to R191, R16 to R192, R15 to R193, R14 to R194, R33 to R195, R67 to R196, R49 to R197, R50 to R198, R51 to R199, R52 to R200, R53 to R201, R54 to R202, R62 to R203, U2 to U10

Commit message: VDD_3V3 is now VDD_3V6 (Removed LDO) LEDs now have the right symbol (oops x2)
Connections:
- net VDD_3V3 renamed VDD_3V6
Changed lines of the file:
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@@
 			)
 		)
-		(property "Value" "VDD_3V3"
+		(property "Value" "VDD_3V6"
 			(at 38.1 38.1 0)
 			(effects
@@
 			)
 		)
-		(property "Value" "VDD_3V3"
+		(property "Value" "VDD_3V6"
 			(at 93.98 118.11 0)
 			(effects
@@
 			)
 		)
-		(property "Value" "VDD_3V3"
+		(property "Value" "VDD_3V6"
 			(at 76.2 163.83 0)
 			(effects
@@
 			)
 		)
-		(property "Value" "VDD_3V3"
+		(property "Value" "VDD_3V6"
 			(at 273.05 46.99 0)
 			(effects
@@
 			)
 		)
-		(property "Value" "VDD_3V3"
+		(property "Value" "VDD_3V6"
 			(at 215.9 76.2 0)
 			(effects

Commit message: Started layout Added some footprints
Parts:
- C67, C68, C69, C70, C73, C74: value 0.1u -> 0u1; footprint Capacitor_SMD:C_0603_1608Metric -> Capacitor_SMD:C_0402_1005Metric
- R196: footprint (none) -> Resistor_SMD:R_0603_1608Metric
Connections:
- net VDD_3V6 renamed VDD_3V3
Changed lines of the file:
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@@
 			)
 		)
-		(property "Footprint" ""
+		(property "Footprint" "Resistor_SMD:R_0603_1608Metric"
 			(at 139.954 86.614 90)
 			(effects
@@
 			)
 		)
-		(property "Value" "VDD_3V6"
+		(property "Value" "VDD_3V3"
 			(at 38.1 38.1 0)
 			(effects
@@
 			)
 		)
-		(property "Value" "0.1u"
+		(property "Value" "0u1"
 			(at 218.44 60.9599 0)
 			(effects
@@
 			)
 		)
-		(property "Footprint" "Capacitor_SMD:C_0603_1608Metric"
+		(property "Footprint" "Capacitor_SMD:C_0402_1005Metric"
 			(at 221.2848 63.5 0)
 			(effects
@@
 			)
 		)
-		(property "Value" "0.1u"
+		(property "Value" "0u1"
 			(at 87.63 165.1 90)
 			(effects
@@
 			)
 		)
-		(property "Footprint" "Capacitor_SMD:C_0603_1608Metric"
+		(property "Footprint" "Capacitor_SMD:C_0402_1005Metric"
 			(at 83.82 171.1452 0)
 			(effects
@@
 			)
 		)
-		(property "Value" "0.1u"
+		(property "Value" "0u1"
 			(at 243.84 60.9599 0)
 			(effects
@@
 			)
 		)
-		(property "Footprint" "Capacitor_SMD:C_0603_1608Metric"
+		(property "Footprint" "Capacitor_SMD:C_0402_1005Metric"
 			(at 246.6848 63.5 0)
 			(effects
@@
 			)
 		)
-		(property "Value" "VDD_3V6"
+		(property "Value" "VDD_3V3"
 			(at 93.98 118.11 0)
 			(effects
@@
 			)
 		)
-		(property "Value" "VDD_3V6"
+		(property "Value" "VDD_3V3"
 			(at 76.2 163.83 0)
 			(effects
@@
 			)
 		)
-		(property "Value" "0.1u"
+		(property "Value" "0u1"
 			(at 256.54 60.9599 0)
 			(effects
@@
 			)
 		)
-		(property "Footprint" "Capacitor_SMD:C_0603_1608Metric"
+		(property "Footprint" "Capacitor_SMD:C_0402_1005Metric"
 			(at 259.3848 63.5 0)
 			(effects
@@
 			)
 		)
-		(property "Value" "0.1u"
+		(property "Value" "0u1"
 			(at 231.14 60.9599 0)
 			(effects
@@
 			)
 		)
-		(property "Footprint" "Capacitor_SMD:C_0603_1608Metric"
+		(property "Footprint" "Capacitor_SMD:C_0402_1005Metric"
 			(at 233.9848 63.5 0)
 			(effects
@@
 			)
 		)
-		(property "Value" "VDD_3V6"
+		(property "Value" "VDD_3V3"
 			(at 273.05 46.99 0)
 			(effects
@@
 			)
 		)
-		(property "Value" "VDD_3V6"
+		(property "Value" "VDD_3V3"
 			(at 215.9 76.2 0)
 			(effects
@@
 			)
 		)
-		(property "Value" "0.1u"
+		(property "Value" "0u1"
 			(at 146.05 166.3699 0)
 			(effects
@@
 			)
 		)
-		(property "Footprint" "Capacitor_SMD:C_0603_1608Metric"
+		(property "Footprint" "Capacitor_SMD:C_0402_1005Metric"
 			(at 143.2052 168.91 0)
 			(effects

Commit message: Added better LIB tree Continued PCB layout Some fixes Added chip for protection
Parts:
- removed J17: Micro_SD_Card_Det1, UserFootprints:GCT_MEM2075-00-140-01-A, symbol Connector:Micro_SD_Card_Det1
- added C111, C112: 0u1, Capacitor_SMD:C_0402_1005Metric, symbol Device:C
- added J17, J32: Micro_SD_Card_Det_Hirose_DM3AT, Connector_Card:microSD_HC_Hirose_DM3AT-SF-PEJM5, symbol Connector:Micro_SD_Card_Det_Hirose_DM3AT
- added R161, R163, R166, R169, R170, R184, R228: 10k, Resistor_SMD:R_0402_1005Metric, symbol Device:R_US
Connections:
- net GND: now also C111.1, C112.2, J17.6 (VSS), J17.9 (DET_B), J32.6 (VSS), J32.9 (DET_B)
- net VDD_3V3: now also C111.2, J17.4 (VDD), J32.4 (VDD), R161.1, R163.1, R166.1, R169.1, R170.1, R184.1, R228.1
- net at C73.1: now also J32.11 (SHIELD)
- net SD_CLK renamed SD1_CLK
- net SD1_CLK: now also J32.5 (CLK)
- net SD_CMD renamed SD1_CMD
- net SD1_CMD: now also J32.3 (CMD)
- net SD_DAT0 renamed SD1_DAT0
- net SD1_DAT0: now also J32.7 (DAT0)
- net SD_DAT1 renamed SD1_DAT1
- net SD1_DAT1: now also J32.8 (DAT1)
- net SD_DAT2 renamed SD1_DAT2
- net SD1_DAT2: now also J32.1 (DAT2)
- net SD_DAT3 renamed SD1_DAT3
- net SD1_DAT3: now also J32.2 (DAT3/CD)
- net SD_DET renamed SD1_DET
- net SD1_DET: now also J32.10 (DET_A)
- new net: C112.1, J17.11 (SHIELD)
- new net SD2_CLK: J17.5 (CLK), R169.2
- new net SD2_CMD: J17.3 (CMD), R170.2
- new net SD2_DAT0: J17.7 (DAT0), R166.2
- new net SD2_DAT1: J17.8 (DAT1), R163.2
- new net SD2_DAT2: J17.1 (DAT2), R228.2
- new net SD2_DAT3: J17.2 (DAT3/CD), R184.2
- new net SD2_DET: J17.10 (DET_A), R161.2
Other:
- note added: "SD CARD #1"
- note added: "SD CARD #2"
- note removed: "SD CARD"
- moved on the sheet: C67, C68, C69, C70, C71, C72, C73, C74, R185, R186, R187, R188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

Commit message: ajout de page root
Parts:
- removed C111, C112, C67, C68, C69, C70, C73, C74: 0u1, Capacitor_SMD:C_0402_1005Metric, symbol Device:C
- removed C71: 10u, Capacitor_SMD:C_0603_1608Metric, symbol Device:C
- removed C72: 2.2u, Capacitor_SMD:C_0603_1608Metric, symbol Device:C
- removed J17, J32: Micro_SD_Card_Det_Hirose_DM3AT, Connector_Card:microSD_HC_Hirose_DM3AT-SF-PEJM5, symbol Connector:Micro_SD_Card_Det_Hirose_DM3AT
- removed R161, R163, R166, R169, R170, R184, R185, R186, R187, R188, R189, R190, R191, R192, R193, R194, R195, R197, R198, R199, R200, R201, R202, R203, R228: 10k, Resistor_SMD:R_0402_1005Metric, symbol Device:R_US
- removed R196: ?, Resistor_SMD:R_0603_1608Metric, symbol Device:R_US
- removed U10: ~, Package_BGA:LFBGA-153_11.5x13mm_Layout14x14_P0.5mm, symbol FSU_LIB:ASFC32G31T3-51BIN
- added C121, C122, C49, C51: 100n, Capacitor_SMD:C_0603_1608Metric, symbol Device:C
- added C50, C58: 10u, Capacitor_SMD:C_0603_1608Metric, symbol Device:C
- added J14, J5: Micro_SD_Card_Det_Hirose_DM3AT, Connector_Card:microSD_HC_Hirose_DM3AT-SF-PEJM5, symbol Connector:Micro_SD_Card_Det_Hirose_DM3AT
- added R100, R55, R57, R59, R61, R63, R74, R75, R76, R78, R79, R99: 22, Resistor_SMD:R_0402_1005Metric, symbol Device:R_US
- added R100, R101, R65, R67, R77, R80, R95, R96, R97, R98 (x2): 10k, Resistor_SMD:R_0402_1005Metric, symbol Device:R_US
Connections:
- net GND: now also C121.2, C122.2, C49.2, C50.2, C51.2, C58.2, J14.6 (VSS), J14.9 (DET_B), J5.6 (VSS), J5.9 (DET_B)
- new net: C121.1, J14.11 (SHIELD)
- new net: J14.1 (DAT2), R55.2, R65.2
- new net: J5.8 (DAT1), R79.2, R98.2
- new net: J5.7 (DAT0), R101.2, R75.2
- new net: J5.3 (CMD), R100.2, R100.2
- new net: J14.3 (CMD), R77.2, R99.2
- new net: C122.1, J5.11 (SHIELD)
- new net: J5.1 (DAT2), R74.2, R80.2
- new net: J5.2 (DAT3/CD), R76.2, R98.2
- new net: J5.5 (CLK), R78.2
- new net: J14.7 (DAT0), R57.2, R95.2
- new net: J14.8 (DAT1), R63.2, R96.2
- new net: J14.2 (DAT3/CD), R59.2, R67.2
- new net: J14.5 (CLK), R61.2
- new net 3V3: C49.1, C50.1, C51.1, C58.1, J14.4 (VDD), J5.4 (VDD), R100.1, R101.1, R65.1, R67.1, R77.1, R80.1, R95.1, R96.1, R97.1, R98.1, R98.1
- new net SD.DET: J14.10 (DET_A), R97.2
- new net SD1.CLK: R61.1
- new net SD1.CMD: R99.1
- new net SD1.DAT0: R57.1
- new net SD1.DAT1: R63.1
- new net SD1.DAT2: R55.1
- new net SD1.DAT3: R59.1
- new net SD2.CLK: R78.1
- new net SD2.CMD: R100.1
- new net SD2.DAT0: R75.1
- new net SD2.DAT1: R79.1
- new net SD2.DAT2: R74.1
- new net SD2.DAT3: R76.1
- new net SD2.DET: J5.10 (DET_A)
Other:
- note removed: "ASFC32G31T3-51BIN"
- note removed: "Impédance match data = 50±5 ohm"
- note removed: "Reference design : https://media.digikey.com/pdf/Data%20Sheets/Octavo%20PDFs/DesigningForFlexibilityAround-EMMC.pdf page 7"
- note removed: "eMMC"
