File: ECU_Geg_trust/ECU_Geg_trust.kicad_pcb (KiCad board)
At the start: 6 copper layers, 98 x 96.9 mm, 321 parts, among them J1 Conn_01x01_Pin, J10 Conn_01x01_Pin, J12 Conn_01x04_Socket, J13 Conn_01x08_Socket, J16 DE9_Socket_MountingHoles, J17 USB_C_Receptacle_USB2.0_man, J2 Micro_SD_Card_Det_Hirose_DM3AT, J25 Conn_01x06_Pin, J3 Micro_SD_Card_Det_Hirose_DM3AT, J4 54-00386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

Commit message: modification de quelques traces
Parts:
- moved R135 34.8 mm to (172.1, 90.3), turned to -90 degrees
Connections:
- R135 pad 2: /BOOT0 -> /NRST
Routing:
- net 6V - A: track 93.7 -> 19.4 mm
- net /MCU_NRST: track 47.0 -> 97.7 mm
- net Net-(J3-DAT1): track 11.6 -> 10.6 mm
