File: ECU_Geg_trust/ECU_Geg_trust.kicad_pcb (KiCad board)
At the start: 6 copper layers, 98 x 96.9 mm, 321 parts, among them J1 Conn_01x01_Pin, J10 Conn_01x01_Pin, J12 Conn_01x04_Socket, J13 Conn_01x08_Socket, J16 DE9_Socket_MountingHoles, J17 USB_C_Receptacle_USB2.0_man, J2 Micro_SD_Card_Det_Hirose_DM3AT, J25 Conn_01x06_Pin, J3 Micro_SD_Card_Det_Hirose_DM3AT, J4 54-00386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

Commit message: En gros aucun ajout depuis le dernier commit... Un ti deplacement de trace parci par la
Other:
- board text added: "3V3"
- board text added: "3V9-A"
- board text added: "5V"
- board text added: "5V-A"
- board text added: "VBAT"
- board text added: "VUSB"
Changed lines of the file:
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@@
 		(tags "capacitor")
 		(property "Reference" "JP1"
-			(at -2.14 0.0375 0)
+			(at -2.3 0.0375 0)
 			(layer "F.SilkS")
 			(effects
@@
 		)
 		(stroke
-			(width 0)
+			(width 0.1)
 			(type solid)
 		)
@@
 		)
 	)
+	(gr_text "VBAT"
+		(at 128.6 132.5 0)
+		(layer "F.SilkS" knockout)
+		(effects
+			(font
+				(size 1 1)
+				(thickness 0.1)
+			)
+			(justify left bottom)
+		)
+	)
 	(gr_text "3V9-A  EN\n"
 		(at 142.5 68.8 90)
@@
 		)
 	)
+	(gr_text "5V-A"
+		(at 128.1 59.5 0)
+		(layer "B.SilkS" knockout)
+		(effects
+			(font
+				(size 1 1)
+				(thickness 0.1)
+			)
+			(justify left bottom mirror)
+		)
+	)
+	(gr_text "VUSB"
+		(at 115.5 117.4 0)
+		(layer "B.SilkS" knockout)
+		(effects
+			(font
+				(size 1 1)
+				(thickness 0.1)
+			)
+			(justify left bottom mirror)
+		)
+	)
 	(gr_text "SIRIUS "
 		(at 151 70.9 0)
@@
 		)
 	)
+	(gr_text "3V3"
+		(at 149.9 94.6 0)
+		(layer "B.SilkS" knockout)
+		(effects
+			(font
+				(size 1 1)
+				(thickness 0.1)
+			)
+			(justify left bottom mirror)
+		)
+	)
+	(gr_text "5V\n"
+		(at 190.2 146.3 0)
+		(layer "B.SilkS" knockout)
+		(effects
+			(font
+				(size 1 1)
+				(thickness 0.1)
+			)
+			(justify left bottom mirror)
+		)
+	)
+	(gr_text "3V9-A\n"
+		(at 156.6 73.2 0)
+		(layer "B.SilkS" knockout)
+		(effects
+			(font
+				(size 1 1)
+				(thickness 0.1)
+			)
+			(justify left bottom mirror)
+		)
+	)
 	(segment
 		(start 156.15 143.21)
@@
 	)
 	(segment
-		(start 126.93 139.32)
-		(end 128.25 140.64)
-		(width 0.2)
-		(layer "B.Cu")
-		(net 166)
-	)
-	(segment
-		(start 129 122.5)
-		(end 130.4 123.9)
+		(start 126.93 136.79)
+		(end 126.93 139.32)
 		(width 0.2)
 		(layer "B.Cu")
@@
 	)
 	(segment
-		(start 128.15 126.15)
-		(end 127.21384 126.15)
+		(start 126.7 126.66384)
+		(end 126.7 129.15)
 		(width 0.2)
 		(layer "B.Cu")
@@
 	)
 	(segment
-		(start 133.15 139.44)
-		(end 133.15 137.47)
+		(start 129 122.5)
+		(end 130.4 123.9)
 		(width 0.2)
 		(layer "B.Cu")
@@
 	)
 	(segment
-		(start 125.6 130.25)
-		(end 125.6 135.46)
+		(start 126.7 129.15)
+		(end 125.6 130.25)
 		(width 0.2)
 		(layer "B.Cu")
@@
 	)
 	(segment
-		(start 136.915192 135.710224)
-		(end 137.993426 134.63199)
+		(start 134.909776 135.710224)
+		(end 136.915192 135.710224)
 		(width 0.2)
 		(layer "B.Cu")
@@
 	)
 	(segment
-		(start 128.25 140.64)
-		(end 128.36 140.53)
+		(start 125.6 130.25)
+		(end 125.6 135.46)
 		(width 0.2)
 		(layer "B.Cu")
@@
 	)
 	(segment
-		(start 132.02 140.53)
-		(end 133.11 139.44)
+		(start 125.6 135.46)
+		(end 126.93 136.79)
 		(width 0.2)
 		(layer "B.Cu")
@@
 	)
 	(segment
-		(start 137.993426 132.133001)
-		(end 137.830814 131.970389)
+		(start 133.3 139.2)
+		(end 133.3 137.32)
 		(width 0.2)
 		(layer "B.Cu")
@@
 	)
 	(segment
-		(start 128.36 140.53)
-		(end 132.02 140.53)
+		(start 128.15 126.15)
+		(end 127.21384 126.15)
 		(width 0.2)
 		(layer "B.Cu")
@@
 	)
 	(segment
-		(start 134.909776 135.710224)
-		(end 136.915192 135.710224)
-		(width 0.2)
-		(layer "B.Cu")
-		(net 166)
-	)
-	(segment
-		(start 127.21384 126.15)
-		(end 126.7 126.66384)
+		(start 133.3 137.32)
+		(end 134.909776 135.710224)
 		(width 0.2)
 		(layer "B.Cu")
@@
 	)
 	(segment
-		(start 126.93 136.79)
-		(end 126.93 139.32)
+		(start 130.4 123.9)
+		(end 128.15 126.15)
 		(width 0.2)
 		(layer "B.Cu")
@@
 	)
 	(segment
-		(start 125.6 135.46)
-		(end 126.93 136.79)
+		(start 137.993426 134.63199)
+		(end 137.993426 132.133001)
 		(width 0.2)
 		(layer "B.Cu")
@@
 	)
 	(segment
-		(start 133.15 137.47)
-		(end 134.909776 135.710224)
+		(start 131.8 140.7)
+		(end 133.3 139.2)
 		(width 0.2)
 		(layer "B.Cu")
@@
 	)
 	(segment
-		(start 126.7 126.66384)
-		(end 126.7 129.15)
+		(start 137.993426 132.133001)
+		(end 137.830814 131.970389)
 		(width 0.2)
 		(layer "B.Cu")
@@
 	)
 	(segment
-		(start 126.7 129.15)
-		(end 125.6 130.25)
+		(start 128.31 140.7)
+		(end 131.8 140.7)
 		(width 0.2)
 		(layer "B.Cu")
@@
 	)
 	(segment
-		(start 130.4 123.9)
-		(end 128.15 126.15)
+		(start 136.915192 135.710224)
+		(end 137.993426 134.63199)
 		(width 0.2)
 		(layer "B.Cu")
@@
 	)
 	(segment
-		(start 133.11 139.44)
-		(end 133.15 139.44)
+		(start 126.93 139.32)
+		(end 128.31 140.7)
 		(width 0.2)
 		(layer "B.Cu")
@@
 	)
 	(segment
-		(start 137.993426 134.63199)
-		(end 137.993426 132.133001)
+		(start 127.21384 126.15)
+		(end 126.7 126.66384)
 		(width 0.2)
 		(layer "B.Cu")

Commit message: Commentaires matis
Routing:
- net /ADS_MOSI: track 9.16 -> 9.92 mm
- net /ADS_MISO: track 8.71 -> 9.27 mm
Other:
- board text added: "Thomas Bélanger Matis Poulin Engine Control Unit Rev 1 Avril 2026"
