File: ECU_Geg_trust/ECU_Geg_trust.kicad_pcb (KiCad board)
At the start: 6 copper layers, 98 x 96.9 mm, 324 parts, among them J1 Conn_01x01_Pin, J10 Conn_01x01_Pin, J12 Conn_01x04_Socket, J13 Conn_01x08_Socket, J16 DE9_Socket_MountingHoles, J17 USB_C_Receptacle_USB2.0_man, J2 Micro_SD_Card_Det_Hirose_DM3AT, J25 Conn_01x06_Pin, J3 Micro_SD_Card_Det_Hirose_DM3AT, J4 54-00386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

Commit message: Reste a faire le BOM
Parts:
- L1, L2, L3: value 1.5uH -> 4u7
Routing:
- net Net-(BT2-+): vias 1 -> 0
