File: ECU_Geg_trust/ECU_Geg_trust.kicad_sch (KiCad schematic)
At the start: 321 parts, among them J1 Conn_01x01_Pin, J10 Conn_01x01_Pin, J12 Conn_01x04_Socket, J13 Conn_01x08_Socket, J16 DE9_Socket_MountingHoles, J17 USB_C_Receptacle_USB2.0_man, J2 Micro_SD_Card_Det_Hirose_DM3AT, J25 Conn_01x06_Pin, J3 Micro_SD_Card_Det_Hirose_DM3AT, J4 54-00386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

Commit message: modification de quelques traces
Connections:
- net BOOT0: no longer R135.2
- net NRST: now also R135.2
Other:
- moved on the sheet: R135
Changed lines of the file:
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@@
 	(wire
 		(pts
+			(xy 697.23 187.96) (xy 697.23 189.23)
+		)
+		(stroke
+			(width 0)
+			(type default)
+		)
+	)
+	(wire
+		(pts
 			(xy 125.73 361.95) (xy 125.73 358.14)
 		)
@@
 	(wire
 		(pts
-			(xy 695.96 166.37) (xy 695.96 165.1)
-		)
-		(stroke
-			(width 0)
-			(type default)
-		)
-	)
-	(wire
-		(pts
 			(xy 566.42 148.59) (xy 566.42 149.86)
 		)
@@
 	(wire
 		(pts
-			(xy 684.53 166.37) (xy 695.96 166.37)
-		)
-		(stroke
-			(width 0)
-			(type default)
-		)
-	)
-	(wire
-		(pts
 			(xy 38.1 351.79) (xy 38.1 360.68)
 		)
@@
 	(wire
 		(pts
-			(xy 295.91 236.22) (xy 307.34 236.22)
+			(xy 290.83 236.22) (xy 307.34 236.22)
 		)
 		(stroke
@@
 	(wire
 		(pts
-			(xy 695.96 156.21) (xy 695.96 157.48)
+			(xy 688.34 265.43) (xy 690.88 265.43)
 		)
 		(stroke
@@
 	(wire
 		(pts
-			(xy 688.34 265.43) (xy 690.88 265.43)
+			(xy 219.71 43.18) (xy 204.47 43.18)
 		)
 		(stroke
@@
 	(wire
 		(pts
-			(xy 219.71 43.18) (xy 204.47 43.18)
+			(xy 521.97 429.26) (xy 529.59 429.26)
 		)
 		(stroke
@@
 	(wire
 		(pts
-			(xy 521.97 429.26) (xy 529.59 429.26)
+			(xy 697.23 198.12) (xy 697.23 196.85)
 		)
 		(stroke
@@
 	(wire
 		(pts
+			(xy 685.8 198.12) (xy 697.23 198.12)
+		)
+		(stroke
+			(width 0)
+			(type default)
+		)
+	)
+	(wire
+		(pts
 			(xy 76.2 48.26) (xy 86.36 48.26)
 		)
@@
 	(wire
 		(pts
-			(xy 295.91 231.14) (xy 320.04 231.14)
+			(xy 290.83 231.14) (xy 320.04 231.14)
 		)
 		(stroke
@@
 	(wire
 		(pts
-			(xy 295.91 233.68) (xy 313.69 233.68)
+			(xy 290.83 233.68) (xy 313.69 233.68)
 		)
 		(stroke
@@
 		)
 	)
-	(label "MCU_NRST"
-		(at 684.53 166.37 0)
-		(effects
-			(font
-				(size 1.27 1.27)
-			)
-			(justify left bottom)
-		)
-	)
 	(label "GPIO5"
 		(at 544.83 414.02 0)
@@
 		)
 	)
+	(label "MCU_NRST"
+		(at 685.8 198.12 0)
+		(effects
+			(font
+				(size 1.27 1.27)
+			)
+			(justify left bottom)
+		)
+	)
 	(label "D+"
 		(at 632.46 113.03 180)
@@
 	)
 	(label "PM_TC"
-		(at 295.91 236.22 0)
+		(at 290.83 236.22 0)
 		(effects
 			(font
@@
 	)
 	(label "PM_CRIT"
-		(at 295.91 231.14 0)
+		(at 290.83 231.14 0)
 		(effects
 			(font
@@
 	)
 	(label "PM_WARN"
-		(at 295.91 233.68 0)
+		(at 290.83 233.68 0)
 		(effects
 			(font
@@
 	(symbol
 		(lib_id "Device:R_US")
-		(at 695.96 161.29 180)
+		(at 697.23 193.04 180)
 		(unit 1)
 		(exclude_from_sim no)
@@
 		(dnp no)
 		(property "Reference" "R135"
-			(at 689.61 159.512 0)
+			(at 690.88 191.262 0)
 			(effects
 				(font
@@
 		)
 		(property "Value" "0"
-			(at 692.912 162.306 0)
+			(at 694.182 194.056 0)
 			(effects
 				(font
@@
 		)
 		(property "Footprint" "Resistor_SMD:R_0603_1608Metric_Pad0.98x0.95mm_HandSolder"
-			(at 694.944 161.036 90)
+			(at 696.214 192.786 90)
 			(effects
 				(font
@@
 		)
 		(property "Datasheet" "~"
-			(at 695.96 161.29 0)
+			(at 697.23 193.04 0)
 			(effects
 				(font
@@
 		)
 		(property "Description" "Resistor, US symbol"
-			(at 695.96 161.29 0)
+			(at 697.23 193.04 0)
 			(effects
 				(font
@@
 		)
 		(property "MANUFACTURER" ""
-			(at 695.96 161.29 0)
+			(at 697.23 193.04 0)
 			(effects
 				(font
@@
 		)
 		(property "MAXIMUM_PACKAGE_HEIGHT" ""
-			(at 695.96 161.29 0)
+			(at 697.23 193.04 0)
 			(effects
 				(font
@@
 		)
 		(property "PARTREV" ""
-			(at 695.96 161.29 0)
+			(at 697.23 193.04 0)
 			(effects
 				(font
@@
 		)
 		(property "STANDARD" ""
-			(at 695.96 161.29 0)
+			(at 697.23 193.04 0)
 			(effects
 				(font
@@
 		)
 		(property "Sim.Device" ""
-			(at 695.96 161.29 0)
+			(at 697.23 193.04 0)
 			(effects
 				(font
@@
 		)
 		(property "Sim.Type" ""
-			(at 695.96 161.29 0)
+			(at 697.23 193.04 0)
 			(effects
 				(font
