File: ECU_Geg_trust/ECU_Geg_trust.kicad_sch (KiCad schematic)
At the start: 323 parts, among them J1 Conn_01x01_Pin, J10 Conn_01x01_Pin, J12 Conn_01x04_Socket, J13 Conn_01x08_Socket, J16 DE9_Socket_MountingHoles, J17 USB_C_Receptacle_USB2.0_man, J2 Micro_SD_Card_Det_Hirose_DM3AT, J25 Conn_01x06_Pin, J3 Micro_SD_Card_Det_Hirose_DM3AT, J4 54-00386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

Commit message: t
Parts:
- U2, U3, U4: value ~ -> (none)

Commit message: BOM pas mal finis reste la valid
Parts:
- BT2: JLCP (none) -> C910763
- C10: value CIN -> 100u; JLCP (none) -> C3344
- C105, C106, C17, C19, C29, C3, C30, C4, C6, C7: value CAP -> 100n; JLCP (none) -> C76997
- C119, C39: JLCP C1592 -> C70225
- C15: value Cdv/dt -> 3n3; JLCP (none) -> C1613
- C28: value C -> 1u; JLCP (none) -> C1592
- C32: value C -> 10u; JLCP (none) -> C3344
- C36, C37: JLCP (none) -> C1592; now left out of the parts list
- C38, C99: JLCP (none) -> C1713
- C64, C81, JP1, JP2, R1, R16, R24, R25, R7, TP2, TP3, TP4, TP5, TP6, TP7: now left out of the parts list
- C78: JLCP (none) -> C1590
- C85: value 0 ohm -> 0
- C87: JLCP (none) -> C115046
- D13: JLCP (none) -> C79598; now left out of the parts list
- F2: JLCP (none) -> C183152
- J1, J10, J12, J8: now not fitted
- J25: now not fitted; now left out of the parts list
- J6: JLCP C17168 -> (none)
- L5: JLCP (none) -> C160977
- R107: value R_US -> 1M; JLCP (none) -> C177344
- R108, R12, R17: value R_US -> 100k; JLCP (none) -> C177329
- R11: value R_US -> 230k; now left out of the parts list
- R15: value R_US -> 400k; now left out of the parts list
- R18: value 1K -> 1k; JLCP (none) -> C22356624
- R19: value RFLT -> 10k; JLCP (none) -> C22369937
- R8: JLCP (none) -> C177329
- R84, R85, R86, R87, R93, R94, R95: value 400 -> 1k; JLCP (none) -> C11702
- U6, U7: JLCP (none) -> C69847
- Y1: JLCP ?? -> C17591433
- Y3: JLCP ?? -> C1987509
