File: ECU_Geg_trust/ECU_Geg_trust.kicad_sch (KiCad schematic)
At the start: 321 parts, among them J1 Conn_01x01_Pin, J10 Conn_01x01_Pin, J12 Conn_01x04_Socket, J13 Conn_01x08_Socket, J16 DE9_Socket_MountingHoles, J17 USB_C_Receptacle_USB2.0_man, J2 Micro_SD_Card_Det_Hirose_DM3AT, J25 Conn_01x06_Pin, J3 Micro_SD_Card_Det_Hirose_DM3AT, J4 54-00386, J5 54-00386, J6 54-00386, J7 54-00386, J8 Conn_01x04_Socket, Q2 BSS138C, SW1 BOOT, SW3 RESET, U1 TPS2595xx, U10 ADS131M04xPW, U11 USBLC6-2SC6, U12 TPS2069CDBV, U13 ISOW1044, U6 LT3042xMSE, U7 LT3042xMSE, U8 INA3221, U9 STM32H747II, Y1 ASV-32.768kHz, Y2 SIT8924BA-22-33E-8.192000, Y3 ASV-25.000MHz

Commit message: Ajout de certain calculs pour eventuellement calculer esl feedback resistors
Other:
- note added: "R = Vout/0.0001"

Commit message: arthur bom
Parts:
- BZ1: JLCP (none) -> C910763
- C1, C104, C59, C60, C62, C65, C66, C69, C83, C84, C85, C91: JLCP (none) -> C76997
- C100, C101, C114, C115, C12, C14, C16, C18, C86, C88, C89, C9, C90, C92, C93, C94, C96, C97: value 0u1 -> 100n; JLCP (none) -> C76997
- C102, C103, C95, C98: JLCP (none) -> C23630
- C107, C20, C31: JLCP (none) -> C1538
- C108, C116, C118, C122, C21, C22, C25, C33, C34, C5, C53, C56: JLCP (none) -> C70225
- C109, C111, C2, C23, C24, C35: JLCP (none) -> C1849
- C11, C120, C52, C54, C55, C57, C61, C70: JLCP (none) -> C1590
- C110, C13, C27: JLCP (none) -> C60425
- C112, C74, C75, C76, C77: value 10n -> 10nF; JLCP (none) -> C1589
- C113: JLCP (none) -> C70225; LCSC (none) -> C1713
- C117, C119, C78, C79: JLCP (none) -> C1592
- C121, C26, C58, C8, C82: value 0u1 -> 100n; JLCP (none) -> C1590
- C38: JLCP (none) -> C1779
- C46, C47, C48, C49, C50, C51: JLCP (none) -> C1872
- C63, C68: JLCP (none) -> C77000
- C67: JLCP (none) -> C23733
- C73: JLCP (none) -> C1589
- C80: JLCP (none) -> C1606
- D1: JLCP (none) -> C5353262
- D10, D4, D5, D6, D7, D8, D9: JLCP (none) -> C2286
- D11: JLCP (none) -> C2891715
- D12, D14: JLCP (none) -> C2500
- D15: JLCP (none) -> C14486
- D2: JLCP (none) -> C82461
- D3: JLCP (none) -> C5656598
- J17: JLCP (none) -> C5184243
- J2, J3: JLCP (none) -> C114218
- J4, J5, J6, J7: JLCP (none) -> C7025199 ps sur
- L1, L2, L3: JLCP (none) -> C2936659 ps sur
- Q2: JLCP (none) -> C255592
- R112, R113: JLCP (none) -> C25905
- R114, R127, R129, R57, R6, R88: JLCP (none) -> C15401
- R128, R37, R39, R41, R45, R47, R48, R60, R61, R62, R63, R64, R65, R96: JLCP (none) -> C159964
- R13, R139, R3: JLCP (none) -> C25545
- R131: JLCP (none) -> C22787
- R138, R14, R4: JLCP (none) -> C26971
- R2, R32, R33, R34, R35, R44, R49, R5, R50, R51, R52, R53, R54, R55, R56, R58, R66, R69: JLCP (none) -> C25531
- R24: now not fitted
- R26, R36: JLCP (none) -> C23193
- R27, R38: JLCP (none) -> C23003
- R28, R40: JLCP (none) -> C25544
- R29, R42: JLCP (none) -> C25818
- R30, R43: JLCP (none) -> C23184
- R31, R46: JLCP (none) -> C156369
- R67, R70: JLCP (none) -> C113041 ps sur
- R71, R73, R74, R75, R76, R77, R78, R79, R80, R81, R82, R83: JLCP (none) -> C14676
- R90, R91, R92: JLCP (none) -> C25530
- SW1, SW3: JLCP (none) -> C2921537
- U1: JLCP (none) -> C471038 ps sur
- U10: JLCP (none) -> C2862562
- U11: JLCP (none) -> C7519
- U12: JLCP (none) -> C181752
- U13: JLCP (none) -> C5216545
- U2, U3: footprint Package_SO:TSSOP-16-1EP_4.4x5mm_P0.65mm_EP3x3mm -> Package_SO:HTSSOP-16-1EP_4.4x5mm_P0.65mm_EP3.4x5mm_Mask2.46x2.31mm_ThermalVias; JLCP (none) -> C580684 vr ps sur
- U4: footprint Package_SO:TSSOP-16_4.4x5mm_P0.65mm -> Package_SO:HTSSOP-16-1EP_4.4x5mm_P0.65mm_EP3.4x5mm_Mask2.46x2.31mm_ThermalVias; JLCP (none) -> C580684 vr ps sur
- U6, U7: JLCP (none) -> C580009 pas sur
- U8: JLCP (none) -> C181255
- U9: JLCP (none) -> C730199
- Y1, Y3: JLCP (none) -> ??
- Y2: JLCP (none) -> C7496633
Connections:
- net GND: no longer U1.9 (GND)
- net at C85.1: now also J4.6; no longer J4.SH
- net at C83.1: now also J7.6; no longer J7.SH
- net at C104.1: now also J5.6; no longer J5.SH
- net at C84.1: now also J6.6; no longer J6.SH

Commit message: arthur
Parts:
- R10, R100, R101, R102, R103, R104, R105, R106, R109, R110, R111, R115, R116, R117, R118, R119, R120, R121, R122, R123, R124, R125, R126, R132, R133, R134, R136, R137, R59, R68, R89, R97, R98, R99: JLCP (none) -> C17168
- R130, R135, R72: JLCP (none) -> C15402
- R9: JLCP (none) -> C158960
Changed lines of the file:
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@@
 			)
 		)
-		(property "JLCP" ""
+		(property "JLCP" "C158960"
 			(at 198.12 40.64 90)
 			(effects
@@
 			)
 		)
-		(property "JLCP" ""
+		(property "JLCP" "C17168"
 			(at 576.58 95.25 90)
 			(effects
@@
 			)
 		)
-		(property "JLCP" ""
+		(property "JLCP" "C17168"
 			(at 655.32 95.25 90)
 			(effects
@@
 			)
 		)
-		(property "JLCP" ""
+		(property "JLCP" "C17168"
 			(at 617.22 97.79 90)
 			(effects
@@
 			)
 		)
-		(property "JLCP" ""
+		(property "JLCP" "C17168"
 			(at 617.22 105.41 90)
 			(effects
@@
 			)
 		)
-		(property "JLCP" ""
+		(property "JLCP" "C17168"
 			(at 655.32 92.71 90)
 			(effects
@@
 			)
 		)
-		(property "JLCP" ""
+		(property "JLCP" "C17168"
 			(at 617.22 92.71 90)
 			(effects
@@
 			)
 		)
-		(property "JLCP" ""
+		(property "JLCP" "C17168"
 			(at 655.32 49.53 90)
 			(effects
@@
 			)
 		)
-		(property "JLCP" ""
+		(property "JLCP" "C15402"
 			(at 758.19 388.62 0)
 			(effects
@@
 			)
 		)
-		(property "JLCP" ""
+		(property "JLCP" "C17168"
 			(at 576.58 92.71 90)
 			(effects
@@
 			)
 		)
-		(property "JLCP" ""
+		(property "JLCP" "C17168"
 			(at 617.22 107.95 90)
 			(effects
@@
 			)
 		)
-		(property "JLCP" ""
+		(property "JLCP" "C17168"
 			(at 576.58 82.55 90)
 			(effects
@@
 			)
 		)
-		(property "JLCP" ""
+		(property "JLCP" "C15402"
 			(at 697.23 193.04 0)
 			(effects
@@
 			)
 		)
-		(property "JLCP" ""
+		(property "JLCP" "C17168"
 			(at 617.22 100.33 90)
 			(effects
@@
 			)
 		)
-		(property "JLCP" ""
+		(property "JLCP" "C17168"
 			(at 617.22 110.49 90)
 			(effects
@@
 			)
 		)
-		(property "JLCP" ""
+		(property "JLCP" "C17168"
 			(at 617.22 118.11 90)
 			(effects
@@
 			)
 		)
-		(property "JLCP" ""
+		(property "JLCP" "C17168"
 			(at 617.22 95.25 90)
 			(effects
@@
 			)
 		)
-		(property "JLCP" ""
+		(property "JLCP" "C17168"
 			(at 655.32 100.33 90)
 			(effects
@@
 			)
 		)
-		(property "JLCP" ""
+		(property "JLCP" "C17168"
 			(at 576.58 85.09 90)
 			(effects
@@
 			)
 		)
-		(property "JLCP" ""
+		(property "JLCP" "C17168"
 			(at 576.58 100.33 90)
 			(effects
@@
 			)
 		)
-		(property "JLCP" ""
+		(property "JLCP" "C17168"
 			(at 576.58 102.87 90)
 			(effects
@@
 			)
 		)
-		(property "JLCP" ""
+		(property "JLCP" "C17168"
 			(at 655.32 57.15 90)
 			(effects
@@
 			)
 		)
-		(property "JLCP" ""
+		(property "JLCP" "C17168"
 			(at 617.22 115.57 90)
 			(effects
@@
 			)
 		)
-		(property "JLCP" ""
+		(property "JLCP" "C17168"
 			(at 617.22 113.03 90)
 			(effects
@@
 			)
 		)
-		(property "JLCP" ""
+		(property "JLCP" "C17168"
 			(at 617.22 52.07 90)
 			(effects
@@
 			)
 		)
-		(property "JLCP" ""
+		(property "JLCP" "C17168"
 			(at 805.18 275.59 90)
 			(effects
@@
 			)
 		)
-		(property "JLCP" ""
+		(property "JLCP" "C17168"
 			(at 655.32 59.69 90)
 			(effects
@@
 			)
 		)
-		(property "JLCP" ""
+		(property "JLCP" "C17168"
 			(at 576.58 105.41 90)
 			(effects
@@
 			)
 		)
-		(property "JLCP" ""
+		(property "JLCP" "C17168"
 			(at 576.58 97.79 90)
 			(effects
@@
 			)
 		)
-		(property "JLCP" ""
+		(property "JLCP" "C17168"
 			(at 617.22 49.53 90)
 			(effects
@@
 			)
 		)
-		(property "JLCP" ""
+		(property "JLCP" "C17168"
 			(at 655.32 52.07 90)
 			(effects
@@
 			)
 		)
-		(property "JLCP" ""
+		(property "JLCP" "C17168"
 			(at 618.49 165.1 90)
 			(effects
@@
 			)
 		)
-		(property "JLCP" ""
+		(property "JLCP" "C17168"
 			(at 576.58 87.63 90)
 			(effects
@@
 			)
 		)
-		(property "JLCP" ""
+		(property "JLCP" "C15402"
 			(at 505.46 406.4 0)
 			(effects
@@
 			)
 		)
-		(property "JLCP" ""
+		(property "JLCP" "C17168"
 			(at 576.58 90.17 90)
 			(effects
@@
 			)
 		)
-		(property "JLCP" ""
+		(property "JLCP" "C17168"
 			(at 617.22 102.87 90)
 			(effects
@@
 			)
 		)
-		(property "JLCP" ""
+		(property "JLCP" "C17168"
 			(at 655.32 62.23 90)
 			(effects
@@
 			)
 		)
-		(property "JLCP" ""
+		(property "JLCP" "C17168"
 			(at 655.32 54.61 90)
 			(effects

Commit message: Commentaires matis
Parts:
- added C39: 10u, Capacitor_SMD:C_0603_1608Metric, symbol Device:C
- added C40: 100nF, Capacitor_SMD:C_0603_1608Metric, symbol Device:C
- C104, C83, C84: value 100n -> 0; JLCP C76997 -> C17168
- C119: value 1u -> 10u
- C38: value 4u7 -> 10u; JLCP C1779 -> (none)
- C71, C72: JLCP (none) -> C9196
- C78: value 1u -> 100n; JLCP C1592 -> (none)
- C85: value 100n -> 0 ohm; JLCP C76997 -> C17168
- F1: value Fuse -> 4A; JLCP (none) -> C187606
- J13: now not fitted
- J16: JLCP (none) -> C183530
- J4, J5, J7: JLCP C7025199 ps sur -> (none); now not fitted
- J6: JLCP C7025199 ps sur -> C17168; now not fitted
- R18: value RILIM -> 1K
- R7: value RVL1 -> 274k
- R8: value RVL2 -> 100k
- U1: JLCP C471038 ps sur -> C471038
- U6, U7: JLCP C580009 pas sur -> (none)
Connections:
- net CHASSIS_CAN: now also C39.1, C40.1
- net at R130.2, U13.12 (VISOOUT), U13.13 (VSIN): now also C39.2, C40.2
Other:
- note added: "1.7A max"
- note added: "Ajouter des condensateurs de découplage sur l'alim des connecteurs"
- note added: "Connecter VREF+ avec VDDA ou ajouter une ferrite"
- note added: "Mettre resistor dans le bom entre pin 6 des connecteur et gnd sinon pas de sheild sur les cables"
- note added: "Pour une alim 11V, les condo devrait être raté au moins 2x ça"
- note added: "Un peu chere comme LDO, pourrait utiliser le TPS7A47 a la place"
- note added: "si voltage <4.5V, can fonctionne pas"
- moved on the sheet: C117, C118, C119, C120, C38, C73, C79, R130

Commit message: Modification de l'ADC pour un autre qui fonctionne
Parts:
- removed U10: ADS131M04xPW, Package_SO:TSSOP-20_4.4x6.5mm_P0.65mm, symbol Analog_ADC:ADS131M04xPW
- added R140: 0, Resistor_SMD:R_0603_1608Metric_Pad0.98x0.95mm_HandSolder, symbol Device:R_US
- added U5: ADS131M08xPBS, Package_QFP:TQFP-32_5x5mm_P0.5mm, symbol Analog_ADC:ADS131M08xPBS
- U2, U3, U4: value ~ -> (none); footprint Package_SO:HTSSOP-16-1EP_4.4x5mm_P0.65mm_EP3.4x5mm_Mask2.46x2.31mm_ThermalVias -> Package_SO:TSSOP-16-1EP_4.4x5mm_P0.65mm_EP3x3mm
Connections:
- net 3V3: now also U5.26 (DVDD)
- net ADC-CLK: now also U5.23 (XTAL1/CLKIN)
- net ADS_CS: now also U5.17 (~{CS})
- net ADS_DRDY: now also U5.18 (~{DRDY})
- net ADS_MISO: now also U5.20 (DOUT)
- net ADS_MOSI: now also U5.21 (DIN)
- net ADS_SCLK: now also U5.19 (SCLK)
- net ADS_SYNC: now also U5.16 (~{SYNC}/~{RESET})
- net GND: now also U5.13 (AGND), U5.25 (DGND), U5.27 (AGND), U5.28 (AGND)
- net VDD_3V9-A: now also U5.14 (REFIN), U5.15 (AVDD)
- net at C85.1: now also J4.SH; no longer J4.6
- net at C83.1: now also J7.SH; no longer J7.6
- net at C76.2, R75.1: now also U5.5 (AIN4P)
- net at BT2.1 (+), C61.2: now also R140.1; no longer U9.8 (VBAT)
- net at C104.1: now also J5.SH; no longer J5.6
- net at C84.1: now also J6.SH; no longer J6.6
- net at C76.1, R76.1: now also U5.6 (AIN4N)
- net at C75.1, R74.1: now also U5.3 (AIN3N)
- net at C74.1, R82.1: now also U5.2 (AIN2N)
- net at C77.1, R78.1: now also U5.7 (AIN5N)
- net at C77.2, R77.1: now also U5.8 (AIN5P)
- net at C74.2, R81.1: now also U5.1 (AIN2P)
- net at C80.2: now also U5.24 (CAP)
- net at C75.2, R73.1: now also U5.4 (AIN3P)
- new net: R140.2, U9.8 (VBAT)
- no-connect marks 105 -> 114
Other:
- moved on the sheet: C80, R91

Commit message: Reste a faire le BOM
Parts:
- C105, C106, C17, C19, C29, C3, C30, C4, C6, C7: JLCP (none) -> C76997
- L1, L2, L3: value 1.5uH -> 4u7; JLCP C2936659 ps sur -> C882054
- R67, R70: JLCP C113041 ps sur -> C177269
- U2, U3, U4: JLCP C580684 vr ps sur -> C684115
- U5: JLCP (none) -> C2685451
- U6, U7: JLCP (none) -> C580011
Changed lines of the file:
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@@
 			)
 		)
-		(property "JLCP" ""
+		(property "JLCP" "C76997"
 			(at 63.5 430.53 0)
 			(hide yes)
@@
 			)
 		)
-		(property "JLCP" ""
+		(property "JLCP" "C76997"
 			(at 74.93 430.53 0)
 			(hide yes)
@@
 			)
 		)
-		(property "JLCP" ""
+		(property "JLCP" "C76997"
 			(at 38.1 430.53 0)
 			(hide yes)
@@
 			)
 		)
-		(property "JLCP" "C580684 vr ps sur"
+		(property "JLCP" "C684115"
 			(at 93.98 222.25 0)
 			(hide yes)
@@
 			)
 		)
-		(property "JLCP" ""
+		(property "JLCP" "C76997"
 			(at 238.76 334.01 0)
 			(hide yes)
@@
 			)
 		)
-		(property "JLCP" "C580684 vr ps sur"
+		(property "JLCP" "C684115"
 			(at 232.41 341.63 0)
 			(hide yes)
@@
 			)
 		)
-		(property "Value" "1.5uH"
+		(property "Value" "4u7"
 			(at 232.41 326.39 90)
 			(show_name no)
@@
 			)
 		)
-		(property "JLCP" "C2936659 ps sur "
+		(property "JLCP" "C882054"
 			(at 232.41 328.93 90)
 			(hide yes)
@@
 			)
 		)
-		(property "JLCP" ""
+		(property "JLCP" "C76997"
 			(at 226.06 334.01 0)
 			(hide yes)
@@
 			)
 		)
-		(property "JLCP" "C580684 vr ps sur"
+		(property "JLCP" "C684115"
 			(at 88.9 341.63 0)
 			(hide yes)
@@
 			)
 		)
-		(property "JLCP" ""
+		(property "JLCP" "C580011"
 			(at 217.17 232.41 0)
 			(hide yes)
@@
 			)
 		)
-		(property "JLCP" "C113041 ps sur"
+		(property "JLCP" "C177269"
 			(at 627.38 408.94 90)
 			(hide yes)
@@
 			)
 		)
-		(property "JLCP" ""
+		(property "JLCP" "C76997"
 			(at 82.55 334.01 0)
 			(hide yes)
@@
 			)
 		)
-		(property "JLCP" ""
+		(property "JLCP" "C580011"
 			(at 217.17 287.02 0)
 			(hide yes)
@@
 			)
 		)
+		(property "JLCP" "C2685451"
+			(at 735.33 284.48 0)
+			(hide yes)
+			(show_name no)
+			(do_not_autoplace no)
+			(effects
+				(font
+					(size 1.27 1.27)
+				)
+			)
+		)
 		(pin "9"
 		)
@@
 			)
 		)
-		(property "Value" "1.5uH"
+		(property "Value" "4u7"
 			(at 88.9 326.39 90)
 			(show_name no)
@@
 			)
 		)
-		(property "JLCP" "C2936659 ps sur "
+		(property "JLCP" "C882054"
 			(at 88.9 328.93 90)
 			(hide yes)
@@
 			)
 		)
-		(property "JLCP" ""
+		(property "JLCP" "C76997"
 			(at 100.33 214.63 0)
 			(hide yes)
@@
 			)
 		)
-		(property "JLCP" ""
+		(property "JLCP" "C76997"
 			(at 95.25 334.01 0)
 			(hide yes)
@@
 			)
 		)
-		(property "JLCP" ""
+		(property "JLCP" "C76997"
 			(at 50.8 430.53 0)
 			(hide yes)
@@
 			)
 		)
-		(property "JLCP" "C113041 ps sur"
+		(property "JLCP" "C177269"
 			(at 627.38 393.7 90)
 			(hide yes)
@@
 			)
 		)
-		(property "JLCP" ""
+		(property "JLCP" "C76997"
 			(at 87.63 214.63 0)
 			(hide yes)
@@
 			)
 		)
-		(property "Value" "1.5uH"
+		(property "Value" "4u7"
 			(at 93.98 207.01 90)
 			(show_name no)
@@
 			)
 		)
-		(property "JLCP" "C2936659 ps sur "
+		(property "JLCP" "C882054"
 			(at 93.98 209.55 90)
 			(hide yes)

Commit message: board commandé
Parts:
- removed C38: 10u, Capacitor_SMD:C_0805_2012Metric, symbol Device:C
- removed J16: DE9_Socket_MountingHoles, Connector_Dsub:DSUB-9_Socket_Horizontal_P2.77x2.84mm_EdgePinOffset4.94mm_Housed_MountingHolesOffset4.94mm, symbol Connector:DE9_Socket_MountingHoles
- added C123: 100n, Capacitor_SMD:C_0402_1005Metric, symbol 0CSL_D1_V1:CAP_7mm_X_2mm
- added C124, C126, C128, C130: 100n, Capacitor_SMD:C_0603_1608Metric, symbol Device:C
- added C125, C127, C129, C131, C132: 10u, Capacitor_SMD:C_0603_1608Metric, symbol Device:C
- added C41: 1u, Capacitor_SMD:C_0603_1608Metric, symbol Device:C
- added D16, D17, D18, D19, D20, D21, D22, D23: PESD5V0S1BA, Diode_SMD:D_SOD-323, symbol Diode:PESD5V0S1UL
- added J18: DE9_Socket_MountingHoles, Connector_Dsub:DSUB-9_Socket_Vertical_P2.77x2.84mm_MountingHoles, symbol Connector:DE9_Socket_MountingHoles
- BT2, J1, J10, J12, J25, J8, R31, R46, TP2, TP3, TP4, TP5, TP6, TP7: now not fitted; now left out of the parts list
- C10: value CIN -> 100u; JLCP (none) -> C7469933
- C100, C101, C114, C115, C12, C14, C16, C18, C59, C65, C69, C86, C88, C89, C9, C90, C92, C93, C94, C96, C97: JLCP C76997 -> C307331
- C102, C103, C95, C98: JLCP C23630 -> C23630
- C104, C83, C84: JLCP C17168 -> C17168
- C105, C106, C17, C19, C29, C3, C30, C4, C6, C7: value CAP -> 100n
- C110, C13, C27: footprint Capacitor_SMD:C_0402_1005Metric -> Capacitor_SMD:C_0603_1608Metric; JLCP C60425 -> C21117
- C112, C73: JLCP C1589 -> C57112
- C117, C79: JLCP C1592 -> C15849
- C119, C39: JLCP C1592 -> C96446
- C120, C40, C70: JLCP C1590 -> C14663
- C15: value Cdv/dt -> 3n3; JLCP (none) -> C1613
- C28: value C -> 1u; JLCP (none) -> C15849
- C32: value C -> 10u; JLCP (none) -> C7469954
- C36, C37, C64, C81, D13, J13, J4, J5, J6, J7, JP1, JP2, R1, R16, R24, R25: now left out of the parts list
- C46, C47, C48, C49, C50, C51: JLCP C1872 -> C29823
- C63, C68: footprint Capacitor_SMD:C_0402_1005Metric -> Capacitor_SMD:C_0603_1608Metric; JLCP C77000 -> C96446; now left out of the parts list
- C67: footprint Capacitor_SMD:C_0603_1608Metric -> Capacitor_SMD:C_0805_2012Metric; JLCP C23733 -> C1779
- C71, C72: footprint Capacitor_SMD:C_1210_3225Metric -> Capacitor_SMD:C_1206_3216Metric; JLCP C9196 -> C9196
- C74, C75, C76, C77: value 10nF -> 330p; JLCP C1589 -> C1664
- C78: footprint Capacitor_SMD:C_0603_1608Metric -> Capacitor_SMD:C_0402_1005Metric; JLCP (none) -> C307331
- C80: JLCP C1606 -> C21120
- C85: value 0 ohm -> 0
- C87: JLCP (none) -> C52923
- C99: JLCP (none) -> C440198
- D1: JLCP C5353262 -> C5353262
- D10, D4, D5, D6, D7, D8, D9: JLCP C2286 -> C2286
- D11: JLCP C2891715 -> C14996
- D15: JLCP C14486 -> C14486
- D2: footprint Diode_SMD:D_SOD-123 -> Diode_SMD:D_SMA; JLCP C82461 -> C14996
- D3: JLCP C5656598 -> C5656598; now not fitted; now left out of the parts list
- F1: JLCP C187606 -> C187606
- F2: JLCP (none) -> C187606
- FID1, FID2, FID3, FID4, H1, H2, H3, H4: now not fitted
- J17: JLCP C5184243 -> C393939
- J2, J3: JLCP C114218 -> C114218
- L1, L2, L3: JLCP C882054 -> C882054
- L5: JLCP (none) -> C160977
- R107: value R_US -> 1M; JLCP (none) -> C22935
- R108: value R_US -> 100k; JLCP (none) -> C25803
- R11, R17: value R_US -> 75k; JLCP (none) -> C23242
- R112, R113: JLCP C25905 -> C25905
- R114, R127, R129, R57, R6, R88: JLCP C15401 -> C25804
- R12: value R_US -> 33k; JLCP (none) -> C4216
- R128, R37, R39, R41, R45, R47, R48, R60, R61, R62, R63, R64, R65, R96: JLCP C159964 -> C25092
- R13, R139, R3: JLCP C25545 -> C25765
- R130, R135, R72: JLCP C15402 -> C21189
- R131: JLCP C22787 -> C22787
- R138, R14, R4: JLCP C26971 -> C25779
- R140: JLCP C15401 -> C21189
- R15: value R_US -> 300k; JLCP (none) -> C23024
- R18: JLCP (none) -> C21190
- R19: JLCP (none) -> C25804
- R2, R32, R33, R34, R35, R44, R49, R5, R50, R51, R52, R53, R54, R55, R56, R58, R66, R69: JLCP C25531 -> C25744
- R26, R36: JLCP C23193 -> C23193
- R27: value 33k2 -> 33k; JLCP C23003 -> C4216
- R28, R40: JLCP C25544 -> C25764
- R29: value 453k -> 220k; JLCP C25818 -> C22961
- R30: value 49k9 -> 33k; JLCP C23184 -> C4216
- R38: value 33k2 -> 100k; JLCP C23003 -> C25803
- R42: value 453k -> 510k; JLCP C25818 -> C23192
- R43: value 49k9 -> 22k; JLCP C23184 -> C31850
- R67, R70: JLCP C177269 -> C23140
- R7: value 274k -> 510k; JLCP (none) -> C23192
- R71, R79, R80, R83: JLCP C14676 -> C21190
- R73, R74, R75, R76, R77, R78, R81, R82: value 1k -> 470; JLCP C14676 -> C23179
- R8: value 100k -> 47k; JLCP (none) -> C25803
- R84, R85, R86, R87, R93, R94, R95: JLCP (none) -> C25117
- R9: JLCP C158960 -> C158960; now not fitted; now left out of the parts list
- R90, R91, R92: JLCP C25530 -> C25741
- SW1, SW3: JLCP C2921537 -> C2921537
- U1: JLCP C471038 -> C471038
- U2, U3, U4: JLCP C684115 -> C684115
- U5: JLCP C2685451 -> C2862610
- U6, U7: JLCP C580011 -> C461518
- U9: JLCP C730199 -> C730199
- Y1: JLCP ?? -> C51822834
- Y2: value SIT8924BA-22-33E-8.192000 -> OCETGLJANF-8.192MHZ; footprint Oscillator:Oscillator_SMD_SiT_PQFN-4Pin_3.2x2.5mm -> Crystal:Crystal_SMD_7050-4Pin_7.0x5.0mm; JLCP C7496633 -> C242206
- Y3: JLCP ?? -> (none); now not fitted; now left out of the parts list
Connections:
- net CAN_N: now also J18.1, J18.2
- net CAN_P: now also J18.6, J18.7
- net CHASSIS_CAN: now also J18.0 (PAD), J18.3, J18.8
- net GND: now also C123.2, C124.2, C125.2, C126.2, C127.2, C128.2, C129.2, C130.2, C131.2, C132.1, C41.2, D16.2 (A), D17.2 (A), D18.2 (A), D19.2 (A), D20.2 (A), D21.2 (A), D22.2 (A), D23.2 (A)
- net IN0+: now also J5.2, D16.1 (K); no longer J5.3
- net IN0-: now also J5.1, D17.1 (K); no longer J5.4
- net IN1+: now also J4.1, D18.1 (K); no longer J4.3
- net IN1-: now also J4.2, D19.1 (K); no longer J4.4
- net IN2+: now also D20.1 (K)
- net IN2-: now also J7.1, D21.1 (K); no longer J7.3
- net IN3+: now also J6.1, D22.1 (K); no longer J6.2
- net IN3-: now also J6.2, D23.1 (K); no longer J6.4
- net VDD_10V-A: now also J4.3, J5.3, J6.3, J7.3, C124.1, C125.1, C126.1, C127.1, C128.1, C129.1, C130.1, C131.1; no longer J4.2, J5.1, J6.1, J7.1
- net VDD_3V9-A: now also C132.2; no longer U5.14 (REFIN)
- new net: C123.1, C41.1, U5.14 (REFIN)
Other:
- note added: "NEED TO VALIDATE VOLTAGE RATING FOR IOs WILL WE FRIE THE STM ?!? ANSWER : YESS, BAD, BAD, BAD WE WILL INDEED FRIE THE STM (CHECK WITH MATIS PCB...?) I WILL NOT CONNECT THE FAULT PIN... -Fine"
- note added: "THIS SYMBOLS NEEDS TO BE VALIDATED BEFORE ACHATS -Done"
- note removed: "Ajouter des condensateurs de découplage sur l'alim des connecteurs"
- note removed: "Connecter VREF+ avec VDDA ou ajouter une ferrite"
- note removed: "Mettre resistor dans le bom entre pin 6 des connecteur et gnd sinon pas de sheild sur les cables"
- note removed: "NEED TO VALIDATE VOLTAGE RATING FOR IOs WILL WE FRIE THE STM ?!? ANSWER : YESS, BAD, BAD, BAD WE WILL INDEED FRIE THE STM (CHECK WITH MATIS PCB...?) I WILL NOT CONNECT THE FAULT PIN..."
- note removed: "Pour une alim 11V, les condo devrait être raté au moins 2x ça"
- note removed: "THIS SYMBOLS NEEDS TO BE VALIDATED BEFORE ACHATS"
- note removed: "Un peu chere comme LDO, pourrait utiliser le TPS7A47 a la place"
- note removed: "si voltage <4.5V, can fonctionne pas"
